File: Hardware/holter.sch (KiCad schematic (older format))
At the start: 170 parts, among them CN1 2TAP, CN2 2TAP, CN3 3TAP, IC1 256kx8, P1 EE_PROG, P2 PROG, SW1 SW_PUSH, U1 TXB0106, U10 TS5A3159, U11 TS5A3159, U12 ESD_PROTECTOR, U13 ESD_PROTECTOR, U14 ESD_PROTECTOR, U15 ESD_PROTECTOR, U16 ESD_PROTECTOR, U17 ESD_PROTECTOR, U18 ESD_PROTECTOR, U19 ESD_PROTECTOR, U2 TXB0106, U20 ESD_PROTECTOR, U21 ESD_PROTECTOR, U22 ESD_PROTECTOR, U23 ESD_PROTECTOR, U29 LIS2DH12, U3 TiWi-uB2, U4 STM32F4x1_64, U5 uSD, U6 ADS1298, U7 USBULC6-2M6, U8 USB2641, U9 OPA379, X1 32768, X2 8MHz, X3 24MHz

Commit message: Power switching optimizations
Parts:
- R36: value 10k -> 100k
Connections:
- wire segments 340 -> 445

Commit message: Charger short circuit fix. Capacitor optimizations.
Parts:
- removed C133: 10uF, symbol C
- C138: value 10uF -> 1uF
- R50: value 10k -> 100k
Connections:
- wire segments 445 -> 337
Other:
- moved on the sheet: C134

Commit message: Footprints, LC filter
Parts:
- C1, C10, C12, C13, C132, C134, C135, C136, C137, C138, C139, C14, C15, C16, C17, C18, C19, C2, C20, C21, C22, C23, C24, C25, C26, C27, C28, C29, C30, C31, C32, C33, C34, C35, C36, C37, C38, C39, C40, C41, C42, C6, C8, C9, CN1, FB10, FB11, FB12, FB13, FB3, FB4, FB5, FB6, FB7, FB8, FB9: footprint (none) -> Capacitors_SMD:C_0402
- FB2: footprint (none) -> Capacitors_SMD:C_0402; TYPE (none) -> BLM15PG100SN1D
- R1, R10, R11, R12, R13, R14, R15, R16, R17, R18, R19, R2, R20, R21, R22, R23, R24, R25, R26, R27, R28, R29, R3, R30, R31, R32, R33, R34, R36, R37, R38, R39, R4, R40, R41, R42, R43, R44, R45, R46, R47, R48, R49, R5, R6, R7, R8, R9: footprint (none) -> Resistors_SMD:R_0402

Commit message: More footprints.
Parts:
- C11: footprint (none) -> Capacitors_SMD:C_0603
- R50, R51, R52, R53, R54, R55, R56, R57, R58, R59, R60, R61, R62, R78, R79, R80, R81, R82, R83, R85: footprint (none) -> Resistors_SMD:R_0402
- U12, U13, U14, U15, U16, U17, U18, U19, U20, U21, U22, U23: footprint (none) -> Capacitors_SMD:C_0402
- U4: footprint (none) -> Housings_QFP:TQFP-64_10x10mm_Pitch0.5mm
- U9: footprint (none) -> TO_SOT_Packages_SMD:SC-70-5
Changed lines of the file:
@@
 EESchema Schematic File Version 2
+LIBS:holter-rescue
 LIBS:power
 LIBS:device
@@
 F 0 "R51" V 14930 1350 40  0000 C CNN
 F 1 "10k" V 14857 1351 40  0000 C CNN
-F 2 "" V 14780 1350 30  0001 C CNN
+F 2 "Resistors_SMD:R_0402" V 14780 1350 30  0001 C CNN
 F 3 "" H 14850 1350 30  0000 C CNN
 	1    14850 1350
@@
 F 0 "U12" H 13250 1700 60  0000 C CNN
 F 1 "ESD_PROTECTOR" H 13350 2030 60  0001 C CNN
-F 2 "" H 13350 1600 60  0001 C CNN
+F 2 "Capacitors_SMD:C_0402" H 13350 1600 60  0001 C CNN
 F 3 "" H 13350 1600 60  0000 C CNN
 	1    13350 1600
@@
 F 0 "R52" V 14930 1950 40  0000 C CNN
 F 1 "10k" V 14857 1951 40  0000 C CNN
-F 2 "" V 14780 1950 30  0001 C CNN
+F 2 "Resistors_SMD:R_0402" V 14780 1950 30  0001 C CNN
 F 3 "" H 14850 1950 30  0000 C CNN
 	1    14850 1950
@@
 F 0 "U13" H 13250 2300 60  0000 C CNN
 F 1 "ESD_PROTECTOR" H 13350 2630 60  0001 C CNN
-F 2 "" H 13350 2200 60  0001 C CNN
+F 2 "Capacitors_SMD:C_0402" H 13350 2200 60  0001 C CNN
 F 3 "" H 13350 2200 60  0000 C CNN
 	1    13350 2200
@@
 F 0 "R53" V 14930 2550 40  0000 C CNN
 F 1 "10k" V 14857 2551 40  0000 C CNN
-F 2 "" V 14780 2550 30  0001 C CNN
+F 2 "Resistors_SMD:R_0402" V 14780 2550 30  0001 C CNN
 F 3 "" H 14850 2550 30  0000 C CNN
 	1    14850 2550
@@
 F 0 "U14" H 13250 2900 60  0000 C CNN
 F 1 "ESD_PROTECTOR" H 13350 3230 60  0001 C CNN
-F 2 "" H 13350 2800 60  0001 C CNN
+F 2 "Capacitors_SMD:C_0402" H 13350 2800 60  0001 C CNN
 F 3 "" H 13350 2800 60  0000 C CNN
 	1    13350 2800
@@
 F 0 "R54" V 14930 3150 40  0000 C CNN
 F 1 "10k" V 14857 3151 40  0000 C CNN
-F 2 "" V 14780 3150 30  0001 C CNN
+F 2 "Resistors_SMD:R_0402" V 14780 3150 30  0001 C CNN
 F 3 "" H 14850 3150 30  0000 C CNN
 	1    14850 3150
@@
 F 0 "U15" H 13250 3500 60  0000 C CNN
 F 1 "ESD_PROTECTOR" H 13350 3830 60  0001 C CNN
-F 2 "" H 13350 3400 60  0001 C CNN
+F 2 "Capacitors_SMD:C_0402" H 13350 3400 60  0001 C CNN
 F 3 "" H 13350 3400 60  0000 C CNN
 	1    13350 3400
@@
 F 0 "R55" V 14930 3750 40  0000 C CNN
 F 1 "10k" V 14857 3751 40  0000 C CNN
-F 2 "" V 14780 3750 30  0001 C CNN
+F 2 "Resistors_SMD:R_0402" V 14780 3750 30  0001 C CNN
 F 3 "" H 14850 3750 30  0000 C CNN
 	1    14850 3750
@@
 F 0 "U16" H 13250 4100 60  0000 C CNN
 F 1 "ESD_PROTECTOR" H 13350 4430 60  0001 C CNN
-F 2 "" H 13350 4000 60  0001 C CNN
+F 2 "Capacitors_SMD:C_0402" H 13350 4000 60  0001 C CNN
 F 3 "" H 13350 4000 60  0000 C CNN
 	1    13350 4000
@@
 F 0 "R56" V 14930 4350 40  0000 C CNN
 F 1 "10k" V 14857 4351 40  0000 C CNN
-F 2 "" V 14780 4350 30  0001 C CNN
+F 2 "Resistors_SMD:R_0402" V 14780 4350 30  0001 C CNN
 F 3 "" H 14850 4350 30  0000 C CNN
 	1    14850 4350
@@
 F 0 "U17" H 13250 4700 60  0000 C CNN
 F 1 "ESD_PROTECTOR" H 13350 5030 60  0001 C CNN
-F 2 "" H 13350 4600 60  0001 C CNN
+F 2 "Capacitors_SMD:C_0402" H 13350 4600 60  0001 C CNN
 F 3 "" H 13350 4600 60  0000 C CNN
 	1    13350 4600
@@
 F 0 "R57" V 14930 4950 40  0000 C CNN
 F 1 "10k" V 14857 4951 40  0000 C CNN
-F 2 "" V 14780 4950 30  0001 C CNN
+F 2 "Resistors_SMD:R_0402" V 14780 4950 30  0001 C CNN
 F 3 "" H 14850 4950 30  0000 C CNN
 	1    14850 4950
@@
 F 0 "U18" H 13250 5300 60  0000 C CNN
 F 1 "ESD_PROTECTOR" H 13350 5630 60  0001 C CNN
-F 2 "" H 13350 5200 60  0001 C CNN
+F 2 "Capacitors_SMD:C_0402" H 13350 5200 60  0001 C CNN
 F 3 "" H 13350 5200 60  0000 C CNN
 	1    13350 5200
@@
 F 0 "R58" V 14930 5550 40  0000 C CNN
 F 1 "10k" V 14857 5551 40  0000 C CNN
-F 2 "" V 14780 5550 30  0001 C CNN
+F 2 "Resistors_SMD:R_0402" V 14780 5550 30  0001 C CNN
 F 3 "" H 14850 5550 30  0000 C CNN
 	1    14850 5550
@@
 F 0 "U19" H 13250 5900 60  0000 C CNN
 F 1 "ESD_PROTECTOR" H 13350 6230 60  0001 C CNN
-F 2 "" H 13350 5800 60  0001 C CNN
+F 2 "Capacitors_SMD:C_0402" H 13350 5800 60  0001 C CNN
 F 3 "" H 13350 5800 60  0000 C CNN
 	1    13350 5800
@@
 F 0 "R59" V 14930 6150 40  0000 C CNN
 F 1 "10k" V 14857 6151 40  0000 C CNN
-F 2 "" V 14780 6150 30  0001 C CNN
+F 2 "Resistors_SMD:R_0402" V 14780 6150 30  0001 C CNN
 F 3 "" H 14850 6150 30  0000 C CNN
 	1    14850 6150
@@
 F 0 "U20" H 13250 6500 60  0000 C CNN
 F 1 "ESD_PROTECTOR" H 13350 6830 60  0001 C CNN
-F 2 "" H 13350 6400 60  0001 C CNN
+F 2 "Capacitors_SMD:C_0402" H 13350 6400 60  0001 C CNN
 F 3 "" H 13350 6400 60  0000 C CNN
 	1    13350 6400
@@
 F 0 "R60" V 14930 6750 40  0000 C CNN
 F 1 "10k" V 14857 6751 40  0000 C CNN
-F 2 "" V 14780 6750 30  0001 C CNN
+F 2 "Resistors_SMD:R_0402" V 14780 6750 30  0001 C CNN
 F 3 "" H 14850 6750 30  0000 C CNN
 	1    14850 6750
@@
 F 0 "U21" H 13250 7100 60  0000 C CNN
 F 1 "ESD_PROTECTOR" H 13350 7430 60  0001 C CNN
-F 2 "" H 13350 7000 60  0001 C CNN
+F 2 "Capacitors_SMD:C_0402" H 13350 7000 60  0001 C CNN
 F 3 "" H 13350 7000 60  0000 C CNN
 	1    13350 7000
@@
 F 0 "R61" V 14930 7350 40  0000 C CNN
 F 1 "470" V 14857 7351 40  0000 C CNN
-F 2 "" V 14780 7350 30  0001 C CNN
+F 2 "Resistors_SMD:R_0402" V 14780 7350 30  0001 C CNN
 F 3 "" H 14850 7350 30  0000 C CNN
 	1    14850 7350
@@
 F 0 "U22" H 13250 7700 60  0000 C CNN
 F 1 "ESD_PROTECTOR" H 13350 8030 60  0001 C CNN
-F 2 "" H 13350 7600 60  0001 C CNN
+F 2 "Capacitors_SMD:C_0402" H 13350 7600 60  0001 C CNN
 F 3 "" H 13350 7600 60  0000 C CNN
 	1    13350 7600
@@
 F 0 "U9" V 10600 1150 39  0000 C CNN
 F 1 "OPA379" H 10800 1150 39  0000 C CNN
-F 2 "" H 10800 1150 39  0001 C CNN
+F 2 "TO_SOT_Packages_SMD:SC-70-5" H 10800 1150 39  0001 C CNN
 F 3 "" H 10800 1150 39  0000 C CNN
 	1    10800 1150
@@
 F 0 "C11" H 8475 4850 30  0000 L CNN
 F 1 "10uF" H 8475 4750 30  0000 L CNN
-F 2 "" H 8450 4800 60  0001 C CNN
+F 2 "Capacitors_SMD:C_0603" H 8450 4800 60  0001 C CNN
 F 3 "" H 8450 4800 60  0000 C CNN
 	1    8450 4800
@@
 F 0 "R50" V 14680 8200 40  0000 C CNN
 F 1 "100k" V 14607 8201 40  0000 C CNN
-F 2 "" V 14530 8200 30  0001 C CNN
+F 2 "Resistors_SMD:R_0402" V 14530 8200 30  0001 C CNN
 F 3 "" H 14600 8200 30  0000 C CNN
 	1    14600 8200
@@
 F 0 "U23" H 13250 8300 60  0000 C CNN
 F 1 "ESD_PROTECTOR" H 13350 8630 60  0001 C CNN
-F 2 "" H 13350 8200 60  0001 C CNN
+F 2 "Capacitors_SMD:C_0402" H 13350 8200 60  0001 C CNN
 F 3 "" H 13350 8200 60  0000 C CNN
 	1    13350 8200
@@
 F 0 "R62" V 15030 7950 40  0000 C CNN
 F 1 "47k" V 14957 7951 40  0000 C CNN
-F 2 "" V 14880 7950 30  0001 C CNN
+F 2 "Resistors_SMD:R_0402" V 14880 7950 30  0001 C CNN
 F 3 "" H 14950 7950 30  0000 C CNN
 	1    14950 7950
@@
 F 0 "U4" H 3350 2750 39  0000 C CNN
 F 1 "STM32F4x1_64" H 3350 2650 39  0000 C CNN
-F 2 "" H 3350 2650 39  0001 C CNN
+F 2 "Housings_QFP:TQFP-64_10x10mm_Pitch0.5mm" H 3350 2650 39  0001 C CNN
 F 3 "" H 3350 2650 39  0000 C CNN
 	1    3350 2650
@@
 F 0 "R78" V 10280 6700 40  0000 C CNN
 F 1 "100" V 10207 6701 40  0000 C CNN
-F 2 "" V 10130 6700 30  0001 C CNN
+F 2 "Resistors_SMD:R_0402" V 10130 6700 30  0001 C CNN
 F 3 "" H 10200 6700 30  0000 C CNN
 	1    10200 6700
@@
 F 0 "R83" V 10630 2000 40  0000 C CNN
 F 1 "10k" V 10557 2001 40  0000 C CNN
-F 2 "" V 10480 2000 30  0001 C CNN
+F 2 "Resistors_SMD:R_0402" V 10480 2000 30  0001 C CNN
 F 3 "" H 10550 2000 30  0000 C CNN
 	1    10550 2000
@@
 F 0 "R79" V 6180 10150 40  0000 C CNN
 F 1 "R" V 6107 10151 40  0000 C CNN
-F 2 "" V 6030 10150 30  0001 C CNN
+F 2 "Resistors_SMD:R_0402" V 6030 10150 30  0001 C CNN
 F 3 "" H 6100 10150 30  0000 C CNN
 	1    6100 10150
@@
 F 0 "R81" V 6380 10150 40  0000 C CNN
 F 1 "R" V 6307 10151 40  0000 C CNN
-F 2 "" V 6230 10150 30  0001 C CNN
+F 2 "Resistors_SMD:R_0402" V 6230 10150 30  0001 C CNN
 F 3 "" H 6300 10150 30  0000 C CNN
 	1    6300 10150
@@
 F 0 "R82" V 6580 10150 40  0000 C CNN
 F 1 "R" V 6507 10151 40  0000 C CNN
-F 2 "" V 6430 10150 30  0001 C CNN
+F 2 "Resistors_SMD:R_0402" V 6430 10150 30  0001 C CNN
 F 3 "" H 6500 10150 30  0000 C CNN
 	1    6500 10150
@@
 F 0 "R80" V 4880 8050 40  0000 C CNN
 F 1 "100k" V 4807 8051 40  0000 C CNN
-F 2 "" V 4730 8050 30  0001 C CNN
+F 2 "Resistors_SMD:R_0402" V 4730 8050 30  0001 C CNN
 F 3 "" H 4800 8050 30  0000 C CNN
 	1    4800 8050
@@
 F 0 "R85" V 14730 8900 40  0000 C CNN
 F 1 "100k" V 14657 8901 40  0000 C CNN
-F 2 "" V 14580 8900 30  0001 C CNN
+F 2 "Resistors_SMD:R_0402" V 14580 8900 30  0001 C CNN
 F 3 "" H 14650 8900 30  0000 C CNN
 	1    14650 8900

Commit message: More footprints.
Parts:
- FB1: footprint (none) -> Capacitors_SMD:C_0603
Changed lines of the file:
@@
 EESchema Schematic File Version 2
-LIBS:holter-rescue
 LIBS:power
 LIBS:device
@@
 F 0 "FB1" H 10300 10800 60  0000 C CNN
 F 1 "MPZ1608D101B (100Ohm @ 100MHz, 1A, 0603)" H 10300 10550 20  0000 C CNN
-F 2 "" H 10300 10650 60  0001 C CNN
+F 2 "Capacitors_SMD:C_0603" H 10300 10650 60  0001 C CNN
 F 3 "" H 10300 10650 60  0000 C CNN
 	1    10300 10650

Commit message: Remove EEPROM programming port
Parts:
- removed P1: EE_PROG, symbol CONN_01X04
Connections:
- wire segments 337 -> 333
Changed lines of the file:
@@
 	1    0    0    -1
 $EndComp
-$Comp
-L GND #PWR0104
-U 1 1 54109C5D
-P 6750 8250
-F 0 "#PWR0104" H 6750 8250 30  0001 C CNN
-F 1 "GND" H 6750 8180 30  0001 C CNN
-F 2 "" H 6750 8250 60  0000 C CNN
-F 3 "" H 6750 8250 60  0000 C CNN
-	1    6750 8250
-	0    -1   -1   0
-$EndComp
-Wire Wire Line
-	6950 7950 6700 7950
-Wire Wire Line
-	6950 6850 6950 7950
 Wire Wire Line
 	6950 6850 7600 6850
@@
 	6950 6700 7000 6700
 Wire Wire Line
-	7000 6700 7000 8050
-Wire Wire Line
-	7000 8050 6700 8050
-Wire Wire Line
 	7600 7050 7050 7050
-Wire Wire Line
-	7050 7050 7050 8150
-Wire Wire Line
-	7050 8150 6700 8150
 $Comp
 L R R30
@@
 Wire Wire Line
 	6750 7350 7050 7350
-Connection ~ 7050 7350
 Wire Wire Line
 	7600 6750 7000 6750
 Connection ~ 7000 6750
-Wire Wire Line
-	6700 8250 6750 8250
 $Comp
 L R R31
@@
 Wire Wire Line
 	6750 7500 7000 7500
-Connection ~ 7000 7500
 Wire Wire Line
 	6750 7650 6950 7650
-Connection ~ 6950 7650
 Connection ~ 8350 5300
 Text GLabel 7600 6100 0    39   BiDi ~ 0
@@
 	1    0    0    -1
 $EndComp
-$Comp
-L CONN_01X04 P1
-U 1 1 54E7C69D
-P 6500 8100
-F 0 "P1" H 6500 8350 50  0000 C CNN
-F 1 "EE_PROG" V 6600 8100 50  0000 C CNN
-F 2 "" H 6500 8100 60  0001 C CNN
-F 3 "" H 6500 8100 60  0000 C CNN
-	1    6500 8100
-	-1   0    0    1
-$EndComp
 Wire Wire Line
 	13750 1400 13750 1350
@@
 Wire Wire Line
 	6300 9150 6950 9150
+Wire Wire Line
+	7000 7500 7000 6700
+Wire Wire Line
+	7050 7350 7050 7050
+Wire Wire Line
+	6950 7650 6950 6850
 $EndSCHEMATC

Commit message: Resistor nets + HTQFP_64 footprint.
Parts:
- removed R1, R12, R13, R14, R15, R16, R17, R9: 100k, Resistors_SMD:R_0402, symbol R
- removed R19, R2, R20, R21, R22, R23, R24, R25, R26, R27, R3, R4, R5, R6, R7: 47, Resistors_SMD:R_0402, symbol R
- added RP? (x2): 51R, symbol R_PACK8
- added RP?: 100k, symbol R_PACK8
Connections:
- wire segments 333 -> 339
- no-connect marks 28 -> 30
Other:
- moved on the sheet: ANT1, CONN1, F1, FB1, R8, U3, U7
