File: Hardware/holter.sch (KiCad schematic (older format))
At the start: 148 parts, among them CN1 2TAP, CN2 2TAP, CN3 3TAP, IC1 256kx8, P2 PROG, SW1 SW_PUSH, U1 TXB0106, U10 TS5A3159, U11 TS5A3159, U12 ESD_PROTECTOR, U13 ESD_PROTECTOR, U14 ESD_PROTECTOR, U15 ESD_PROTECTOR, U16 ESD_PROTECTOR, U17 ESD_PROTECTOR, U18 ESD_PROTECTOR, U19 ESD_PROTECTOR, U2 TXB0106, U20 ESD_PROTECTOR, U21 ESD_PROTECTOR, U22 ESD_PROTECTOR, U23 ESD_PROTECTOR, U29 LIS2DH12, U3 TiWi-uB2, U4 STM32F4x1_64, U5 uSD, U6 ADS1298, U7 USBULC6-2M6, U8 USB2641, U9 OPA379, X1 32768, X2 8MHz, X3 24MHz

Commit message: Rearrangement.
Parts:
- removed C136: 1uF, Capacitors_SMD:C_0402, symbol C_Small
- RP? (x2): value 51R -> 51R EXB2HV510JV
- RP?: value 100k -> 100k EXB2HV104JV
Connections:
- wire segments 339 -> 338
Other:
- moved on the sheet: C132, IC1, R30, R31, R32, R33, R35, R36, R78, R80, SW1, U1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

Commit message: Fixed ADS1298 library.
Parts:
- gave numbers to parts that had none: 3
Connections:
- no-connect marks 30 -> 31
Other:
- moved on the sheet: IC1, R30, R31, R32, R33, R35, R36, R78, U8

Commit message: More footprints.
Parts:
- F1: footprint (none) -> Capacitors_SMD:C_1206
- IC1: footprint SOT23-5 -> TO_SOT_Packages_SMD:SOT-23-5
- U10, U11: footprint (none) -> Housings_SOT-23_SOT-143_TSOT-6:SOT-23-6
- U8: footprint (none) -> Housings_DFN_QFN:QFN-48-1EP_7x7mm_Pitch0.5mm
Connections:
- no-connect marks 31 -> 34

Commit message: MicroSD connector pdf, Level shifter QFN -> TSSOP
Parts:
- removed D9: RGBLED, symbol RGBLED
- added LED1, LED2, LED3: LED, LEDs:LED-3MM, symbol LED
- U1, U2: footprint (none) -> Housings_SSOP:TSSOP-16_4.4x5mm_Pitch0.65mm
- U6: footprint (none) -> Footprints:HTQFP_64
Connections:
- wire segments 338 -> 341

Commit message: Footprints...
Parts:
- C7: footprint (none) -> Capacitors_SMD:C_0603
- U29: footprint (none) -> Footprints:LGA12
- U3: footprint (none) -> Footprints:TIWIUB2
- U5: footprint (none) -> Footprints:MEM2051
- U7: footprint (none) -> Footprints:USBULC62M6
Connections:
- no-connect marks 34 -> 38
Changed lines of the file:
@@
 F 0 "C7" H 8025 4850 30  0000 L CNN
 F 1 "22uF" H 8025 4750 30  0000 L CNN
-F 2 "" H 8000 4800 60  0001 C CNN
+F 2 "Capacitors_SMD:C_0603" H 8000 4800 60  0001 C CNN
 F 3 "" H 8000 4800 60  0000 C CNN
 	1    8000 4800
@@
 F 0 "U3" H 3975 10475 39  0000 C CNN
 F 1 "TiWi-uB2" H 4075 10375 39  0000 C CNN
-F 2 "" H 4100 11200 39  0001 C CNN
+F 2 "Footprints:TIWIUB2" H 4100 11200 39  0001 C CNN
 F 3 "" H 4100 11200 39  0000 C CNN
 	1    3750 9900
@@
 F 0 "U5" H 4900 7150 39  0000 C CNN
 F 1 "uSD" V 5200 6750 39  0000 C CNN
-F 2 "" H 5200 6750 39  0001 C CNN
+F 2 "Footprints:MEM2051" H 5200 6750 39  0001 C CNN
 F 3 "" H 5200 6750 39  0000 C CNN
 	1    5050 6750
@@
 F 0 "U7" H 9500 10325 39  0000 C CNN
 F 1 "USBULC6-2M6" H 9500 9875 39  0000 C CNN
-F 2 "" H 8975 11050 39  0001 C CNN
+F 2 "Footprints:USBULC62M6" H 8975 11050 39  0001 C CNN
 F 3 "" H 8975 11050 39  0000 C CNN
 	1    9500 10100
@@
 F 0 "U29" V 13800 9400 39  0000 C CNN
 F 1 "LIS2DH12" V 13900 9400 39  0000 C CNN
-F 2 "" H 13850 10450 39  0001 C CNN
+F 2 "Footprints:LGA12" H 13850 10450 39  0001 C CNN
 F 3 "" H 13850 10450 39  0000 C CNN
 	1    13950 9400
@@
 Wire Wire Line
 	6100 9150 6100 9350
+NoConn ~ 4100 9100
+NoConn ~ 4200 9100
+NoConn ~ 4000 9100
+$Comp
+L GND #PWR0160
+U 1 1 561B3FCF
+P 5700 7050
+F 0 "#PWR0160" H 5700 7050 30  0001 C CNN
+F 1 "GND" H 5700 6980 30  0001 C CNN
+F 2 "" H 5700 7050 60  0000 C CNN
+F 3 "" H 5700 7050 60  0000 C CNN
+	1    5700 7050
+	0    -1   -1   0
+$EndComp
+$Comp
+L GND #PWR0161
+U 1 1 561B46CA
+P 5700 6950
+F 0 "#PWR0161" H 5700 6950 30  0001 C CNN
+F 1 "GND" H 5700 6880 30  0001 C CNN
+F 2 "" H 5700 6950 60  0000 C CNN
+F 3 "" H 5700 6950 60  0000 C CNN
+	1    5700 6950
+	0    -1   -1   0
+$EndComp
+$Comp
+L GND #PWR0162
+U 1 1 561B488B
+P 5700 6850
+F 0 "#PWR0162" H 5700 6850 30  0001 C CNN
+F 1 "GND" H 5700 6780 30  0001 C CNN
+F 2 "" H 5700 6850 60  0000 C CNN
+F 3 "" H 5700 6850 60  0000 C CNN
+	1    5700 6850
+	0    -1   -1   0
+$EndComp
+$Comp
+L GND #PWR0163
+U 1 1 561B4A4C
+P 5700 6750
+F 0 "#PWR0163" H 5700 6750 30  0001 C CNN
+F 1 "GND" H 5700 6680 30  0001 C CNN
+F 2 "" H 5700 6750 60  0000 C CNN
+F 3 "" H 5700 6750 60  0000 C CNN
+	1    5700 6750
+	0    -1   -1   0
+$EndComp
+NoConn ~ 5700 6450
 $EndSCHEMATC

Commit message: Footprints.
Parts:
- C3, C4, R35: footprint (none) -> Capacitors_SMD:C_0402
- C5: footprint (none) -> Capacitors_SMD:C_0603
Changed lines of the file:
@@
 F 0 "C5" V 3950 3750 30  0000 L CNN
 F 1 "4.7uF LOW ESR" V 4000 3450 30  0000 L CNN
-F 2 "" H 3900 3850 60  0001 C CNN
+F 2 "Capacitors_SMD:C_0603" H 3900 3850 60  0001 C CNN
 F 3 "" H 3900 3850 60  0000 C CNN
 	1    3900 3850
@@
 F 0 "C3" H 1075 2100 30  0000 L CNN
 F 1 " C_Small" H 1075 2000 30  0000 L CNN
-F 2 "" H 1050 2050 60  0001 C CNN
+F 2 "Capacitors_SMD:C_0402" H 1050 2050 60  0001 C CNN
 F 3 "" H 1050 2050 60  0000 C CNN
 	1    1050 2050
@@
 F 0 "C4" H 1075 2700 30  0000 L CNN
 F 1 " C_Small" H 1075 2600 30  0000 L CNN
-F 2 "" H 1050 2650 60  0001 C CNN
+F 2 "Capacitors_SMD:C_0402" H 1050 2650 60  0001 C CNN
 F 3 "" H 1050 2650 60  0000 C CNN
 	1    1050 2650
@@
 F 0 "R35" V 8880 8300 40  0000 C CNN
 F 1 "12k 1%" V 8800 8300 40  0000 C CNN
-F 2 "" V 8730 8300 30  0001 C CNN
+F 2 "Capacitors_SMD:C_0402" V 8730 8300 30  0001 C CNN
 F 3 "" H 8800 8300 30  0000 C CNN
 	1    8800 8300

Commit message: Footprints...
Parts:
- ANT1: footprint (none) -> Footprints:2450AT42A100
- CN1: footprint Capacitors_SMD:C_0402 -> Resistors_SMD:R_0402
- CN2: footprint (none) -> Resistors_SMD:R_0402
Connections:
- no-connect marks 38 -> 39
Changed lines of the file:
@@
 F 0 "CN1" H 10850 3050 60  0001 C CNN
 F 1 "2TAP" H 10850 2950 60  0001 C CNN
-F 2 "Capacitors_SMD:C_0402" H 10850 2800 60  0001 C CNN
+F 2 "Resistors_SMD:R_0402" H 10850 2800 60  0001 C CNN
 F 3 "" H 10850 2800 60  0000 C CNN
 	1    10850 2800
@@
 F 0 "CN2" H 10850 3800 60  0001 C CNN
 F 1 "2TAP" H 10850 3700 60  0001 C CNN
-F 2 "" H 10850 3550 60  0001 C CNN
+F 2 "Resistors_SMD:R_0402" H 10850 3550 60  0001 C CNN
 F 3 "" H 10850 3550 60  0000 C CNN
 	1    10850 3550
@@
 U 1 1 540C4324
 P 5050 9300
-F 0 "ANT1" H 5050 9500 39  0000 C CNN
+F 0 "ANT1" H 4850 9350 39  0000 C CNN
 F 1 "2450AT42A100" H 5050 9100 39  0000 C CNN
-F 2 "" H 5000 9670 39  0001 C CNN
+F 2 "Footprints:2450AT42A100" H 5000 9670 39  0001 C CNN
 F 3 "" H 5000 9670 39  0000 C CNN
 	1    5050 9300
@@
 U 1 1 540B179F
 P 3750 9900
-F 0 "U3" H 3975 10475 39  0000 C CNN
-F 1 "TiWi-uB2" H 4075 10375 39  0000 C CNN
+F 0 "U3" H 3650 10450 39  0000 C CNN
+F 1 "TiWi-uB2" H 3350 10050 39  0000 C CNN
 F 2 "Footprints:TIWIUB2" H 4100 11200 39  0001 C CNN
 F 3 "" H 4100 11200 39  0000 C CNN
@@
 $EndComp
 NoConn ~ 5700 6450
+NoConn ~ 5050 8950
 $EndSCHEMATC

Commit message: Footprints.
Parts:
- added P1: CONN_01X05, symbol CONN_01X05
- CONN1: footprint (none) -> Footprints:HDMI10029449
- RP1, RP2, RP3: footprint (none) -> Footprints:EXB2HV
- SW1: footprint (none) -> Footprints:MCTA3
Connections:
- wire segments 341 -> 342
Changed lines of the file:
@@
 F 0 "CONN1" H 8500 11300 39  0000 C CNN
 F 1 "HDMI" H 8500 11350 39  0000 C CNN
-F 2 "" H 8350 10200 39  0001 C CNN
+F 2 "Footprints:HDMI10029449" H 8350 10200 39  0001 C CNN
 F 3 "" H 8350 10200 39  0000 C CNN
 	1    8350 10200
@@
 L GND #PWR0122
 U 1 1 5411DB10
-P 8900 10350
-F 0 "#PWR0122" H 8900 10350 30  0001 C CNN
-F 1 "GND" H 8900 10280 30  0001 C CNN
-F 2 "" H 8900 10350 60  0000 C CNN
-F 3 "" H 8900 10350 60  0000 C CNN
-	1    8900 10350
-	0    -1   -1   0
+P 8900 10550
+F 0 "#PWR0122" H 8900 10550 30  0001 C CNN
+F 1 "GND" H 8900 10480 30  0001 C CNN
+F 2 "" H 8900 10550 60  0000 C CNN
+F 3 "" H 8900 10550 60  0000 C CNN
+	1    8900 10550
+	1    0    0    -1
 $EndComp
 Text GLabel 9750 10250 2    39   BiDi ~ 0
@@
 P 4800 7850
 F 0 "SW1" H 4950 7960 50  0000 C CNN
-F 1 "SW_PUSH" H 4800 7770 50  0000 C CNN
-F 2 "" H 4800 7850 60  0001 C CNN
+F 1 "SW_PUSH" H 4800 8050 50  0000 C CNN
+F 2 "Footprints:MCTA3" H 4800 7850 60  0001 C CNN
 F 3 "" H 4800 7850 60  0000 C CNN
 	1    4800 7850
@@
 F 0 "RP3" H 6200 3850 50  0000 C CNN
 F 1 "51R EXB2HV510JV" H 6100 2900 50  0000 C CNN
-F 2 "" H 6200 3400 60  0001 C CNN
+F 2 "Footprints:EXB2HV" H 6200 3400 60  0001 C CNN
 F 3 "" H 6200 3400 60  0000 C CNN
 	1    6200 3400
@@
 F 0 "RP2" H 3850 6450 50  0000 C CNN
 F 1 "100k EXB2HV104JV" V 3300 6000 50  0000 C CNN
-F 2 "" H 3850 6000 60  0001 C CNN
+F 2 "Footprints:EXB2HV" H 3850 6000 60  0001 C CNN
 F 3 "" H 3850 6000 60  0000 C CNN
 	1    3850 6000
@@
 F 0 "RP1" H 2150 10250 50  0000 C CNN
 F 1 "51R EXB2HV510JV" H 1950 9250 50  0000 C CNN
-F 2 "" H 2150 9800 60  0001 C CNN
+F 2 "Footprints:EXB2HV" H 2150 9800 60  0001 C CNN
 F 3 "" H 2150 9800 60  0000 C CNN
 	1    2150 9800
@@
 NoConn ~ 5700 6450
 NoConn ~ 5050 8950
+Wire Wire Line
+	8900 10300 8900 10550
+Connection ~ 8900 10350
+Connection ~ 8900 10400
+Connection ~ 8900 10450
+$Comp
+L GND #PWR0164
+U 1 1 561DA1CA
+P 4700 8250
+F 0 "#PWR0164" H 4700 8250 30  0001 C CNN
+F 1 "GND" H 4700 8180 30  0001 C CNN
+F 2 "" H 4700 8250 60  0000 C CNN
+F 3 "" H 4700 8250 60  0000 C CNN
+	1    4700 8250
+	1    0    0    -1
+$EndComp
+$Comp
+L GND #PWR0165
+U 1 1 561DA38B
+P 4800 8250
+F 0 "#PWR0165" H 4800 8250 30  0001 C CNN
+F 1 "GND" H 4800 8180 30  0001 C CNN
+F 2 "" H 4800 8250 60  0000 C CNN
+F 3 "" H 4800 8250 60  0000 C CNN
+	1    4800 8250
+	1    0    0    -1
+$EndComp
+$Comp
+L GND #PWR0166
+U 1 1 561DA54C
+P 4900 8250
+F 0 "#PWR0166" H 4900 8250 30  0001 C CNN
+F 1 "GND" H 4900 8180 30  0001 C CNN
+F 2 "" H 4900 8250 60  0000 C CNN
+F 3 "" H 4900 8250 60  0000 C CNN
+	1    4900 8250
+	1    0    0    -1
+$EndComp
+$Comp
+L CONN_01X05 P1
+U 1 1 561DFA81
+P 7350 10450
+F 0 "P1" H 7350 10750 50  0000 C CNN
+F 1 "CONN_01X05" V 7450 10450 50  0000 C CNN
+F 2 "" H 7350 10450 60  0001 C CNN
+F 3 "" H 7350 10450 60  0000 C CNN
+	1    7350 10450
+	1    0    0    -1
+$EndComp
 $EndSCHEMATC
