File: Hardware/holter.sch (KiCad schematic (older format))
At the start: 150 parts, among them CN1 2TAP, CN2 2TAP, CN3 3TAP, IC1 256kx8, P1 CONN_01X05, P2 PROG, SW1 SW_PUSH, U1 TXB0106, U10 TS5A3159, U11 TS5A3159, U12 ESD_PROTECTOR, U13 ESD_PROTECTOR, U14 ESD_PROTECTOR, U15 ESD_PROTECTOR, U16 ESD_PROTECTOR, U17 ESD_PROTECTOR, U18 ESD_PROTECTOR, U19 ESD_PROTECTOR, U2 TXB0106, U20 ESD_PROTECTOR, U21 ESD_PROTECTOR, U22 ESD_PROTECTOR, U23 ESD_PROTECTOR, U29 LIS2DH12, U3 TiWi-uB2, U4 STM32F4x1_64, U5 uSD, U6 ADS1298, U7 USBULC6-2M6, U8 USB2641, U9 OPA379, X1 32768, X2 8MHz, X3 24MHz

Commit message: Footprints.
Parts:
- removed LED1, LED2, LED3: LED, LEDs:LED-3MM, symbol LED
- removed R79: R, Resistors_SMD:R_0402, symbol R
- removed SW1: SW_PUSH, Footprints:MCTA3, symbol SW_PUSH
Connections:
- net labels added: BAT+
- wire segments 342 -> 336
Other:
- moved on the sheet: C132, C134, R80, R81, R82

Commit message: Footprints.
Parts:
- removed X2: 8MHz, symbol Crystal
- removed X3: 24MHz, symbol Crystal
- added Y1: 24 MHz, Footprints:TSX3225, symbol Crystal_4PAD
- added Y2: 10 MHz, Footprints:TSX3225, symbol Crystal_4PAD
- CN3: footprint (none) -> Footprints:SOLDERJUMPER3
- P2: footprint (none) -> Footprints:HEADER127_4
- X1: footprint (none) -> Footprints:FC135
Connections:
- wire segments 336 -> 331
Other:
- moved on the sheet: C134, R33

Commit message: Footprints.
Parts:
- removed P1: CONN_01X05, symbol CONN_01X05
- added P1: CONN_01X07, Footprints:MOBO9155, symbol CONN_01X07
- U1, U2: footprint Housings_SSOP:TSSOP-16_4.4x5mm_Pitch0.65mm -> Footprints:RGY16

Commit message: Outline drawings.
Parts:
- CONN1: footprint Footprints:HDMI10029449 -> Footprints:MC34931
Other:
- moved on the sheet: C132, C134, R80, R81, R82

Commit message: Grounding point, LC filter at 1.8V supply
Parts:
- CONN1: footprint Footprints:MC34931 -> Footprints:2013978
Connections:
- net labels removed: B_PWM
- no-connect marks 39 -> 40
Changed lines of the file:
@@
 F 0 "CONN1" H 8500 11300 39  0000 C CNN
 F 1 "HDMI" H 8500 11350 39  0000 C CNN
-F 2 "Footprints:MC34931" H 8350 10200 39  0001 C CNN
+F 2 "Footprints:2013978" H 8350 10200 39  0001 C CNN
 F 3 "" H 8350 10200 39  0000 C CNN
 	1    8350 10200
@@
 Text GLabel 3100 1450 1    39   Output ~ 0
 G_PWM
-Text GLabel 2900 1450 1    39   Output ~ 0
-B_PWM
 $Comp
 L +2.8VD #PWR0129
@@
 	1    0    0    -1
 $EndComp
-Wire Wire Line
-	6700 9700 7000 9700
-Text Label 6700 9700 0    60   ~ 0
-BAT+
 $Comp
 L Crystal_4PAD Y1
@@
 	0    1    1    0
 $EndComp
+Wire Wire Line
+	7000 9700 6700 9700
+NoConn ~ 2900 1450
+Text GLabel 6700 9700 0    60   Input ~ 0
+BAT+
 $EndSCHEMATC

Commit message: Placement of the I/O filtering components
Parts:
- added R1, R2: 1k, Resistors_SMD:R_0402, symbol R
Connections:
- wire segments 331 -> 334
- no-connect marks 40 -> 38
Changed lines of the file:
@@
 	1    0    0    -1
 $EndComp
-NoConn ~ 9050 4500
 $Comp
 L C C42
@@
 	1    0    0    -1
 $EndComp
-NoConn ~ 9150 4500
 $Comp
 L GND #PWR039
@@
 Connection ~ 9800 1850
 Wire Wire Line
-	10100 1850 10100 3050
+	10100 1850 10100 4500
 Wire Wire Line
 	10550 2150 10550 3800
@@
 Wire Wire Line
 	7000 9700 6700 9700
-NoConn ~ 2900 1450
 Text GLabel 6700 9700 0    60   Input ~ 0
 BAT+
+$Comp
+L R R2
+U 1 1 56268D65
+P 9450 4500
+F 0 "R2" V 9530 4500 40  0000 C CNN
+F 1 "1k" V 9457 4501 40  0000 C CNN
+F 2 "Resistors_SMD:R_0402" V 9380 4500 30  0001 C CNN
+F 3 "" H 9450 4500 30  0000 C CNN
+	1    9450 4500
+	0    1    1    0
+$EndComp
+$Comp
+L R R1
+U 1 1 56268F41
+P 9050 4750
+F 0 "R1" V 9150 4800 40  0000 C CNN
+F 1 "1k" V 9057 4751 40  0000 C CNN
+F 2 "Resistors_SMD:R_0402" V 8980 4750 30  0001 C CNN
+F 3 "" H 9050 4750 30  0000 C CNN
+	1    9050 4750
+	-1   0    0    1
+$EndComp
+$Comp
+L GND #PWR0169
+U 1 1 562692D8
+P 9050 4900
+F 0 "#PWR0169" H 9050 4900 30  0001 C CNN
+F 1 "GND" H 9050 4830 30  0001 C CNN
+F 2 "" H 9050 4900 60  0000 C CNN
+F 3 "" H 9050 4900 60  0000 C CNN
+	1    9050 4900
+	1    0    0    -1
+$EndComp
+Wire Wire Line
+	9050 4600 9050 4500
+Wire Wire Line
+	9150 4500 9300 4500
+Wire Wire Line
+	10100 4500 9600 4500
+Connection ~ 10100 3050
+NoConn ~ 2900 1450
 $EndSCHEMATC

Commit message: Component placement + add 3.3V enable pin
Connections:
- net labels added: EN_3V3
- no-connect marks 38 -> 37
Changed lines of the file:
@@
 	10100 4500 9600 4500
 Connection ~ 10100 3050
-NoConn ~ 2900 1450
+Text GLabel 2900 1450 1    39   Input ~ 0
+EN_3V3
 $EndSCHEMATC

Commit message: USB charger and power supply is now a separate module
Parts:
- added P3: SCREW, Footprints:M2_SCREW, symbol CONN_01X01
Changed lines of the file:
@@
 LIBS:rgbled
 LIBS:lis2dh12
+LIBS:usb_power_module
 LIBS:holter-cache
 EELAYER 25 0
@@
 $Descr A3 16535 11693
 encoding utf-8
-Sheet 1 2
+Sheet 1 3
 Title "MobilECG II"
 Date "sept 1, 2014"
@@
 NoConn ~ 7150 2750
 NoConn ~ 7150 2850
-NoConn ~ 7150 3050
 $Comp
 L C_Small C10
@@
 F 3 "" H 3850 6000 60  0000 C CNN
 	1    3850 6000
-	0    1    1    0
+	0    -1   -1   0
 $EndComp
 $Comp
@@
 Text GLabel 2900 1450 1    39   Input ~ 0
 EN_3V3
+NoConn ~ 7150 3050
+$Comp
+L CONN_01X01 P3
+U 1 1 5627B2F6
+P 6400 5500
+F 0 "P3" H 6400 5600 50  0000 C CNN
+F 1 "SCREW" V 6500 5500 50  0000 C CNN
+F 2 "Footprints:M2_SCREW" H 6400 5500 60  0001 C CNN
+F 3 "" H 6400 5500 60  0000 C CNN
+	1    6400 5500
+	0    -1   -1   0
+$EndComp
+$Comp
+L GND #PWR0170
+U 1 1 5627B8D3
+P 6400 5700
+F 0 "#PWR0170" H 6400 5700 30  0001 C CNN
+F 1 "GND" H 6400 5630 30  0001 C CNN
+F 2 "" H 6400 5700 60  0000 C CNN
+F 3 "" H 6400 5700 60  0000 C CNN
+	1    6400 5700
+	1    0    0    -1
+$EndComp
 $EndSCHEMATC
