File: Hardware/power.sch (KiCad schematic (older format))
At the start: 131 parts, among them P3 BAT+, P4 BAT-, Q1 SI1403, Q2 SI1403, Q3 SI1403, Q4 SI1403, Q5 SI1403, U24 TLV61220, U25 TLV61220, U26 TLV61220, U27 LM3671, U28 DS2710

Commit message: Power switching optimizations
Parts:
- removed D2, D5: D_Schottky, symbol D_Schottky
- removed R84: 100k, symbol R
Connections:
- wire segments 222 -> 214
Changed lines of the file:
@@
 LIBS:rgbled
 LIBS:lis2dh12
+LIBS:holter-cache
 EELAYER 25 0
 EELAYER END
@@
 	6400 5000 6400 5350
 Wire Wire Line
-	6400 5350 8450 5350
+	8450 5350 6400 5350
 Wire Wire Line
-	8450 5350 8450 4550
+	8450 4550 8450 5350
 Wire Wire Line
 	8450 4550 8300 4550
@@
 Connection ~ 3800 4700
 $Comp
-L D_Schottky D5
-U 1 1 541462CE
-P 2200 4050
-F 0 "D5" H 2200 4150 40  0000 C CNN
-F 1 "D_Schottky" H 2200 3950 40  0000 C CNN
-F 2 "" H 2200 4050 60  0000 C CNN
-F 3 "" H 2200 4050 60  0000 C CNN
-	1    2200 4050
-	1    0    0    -1
-$EndComp
-$Comp
 L D_Schottky D3
 U 1 1 541462EE
-P 2200 3750
-F 0 "D3" H 2200 3850 40  0000 C CNN
-F 1 "D_Schottky" H 2200 3650 40  0000 C CNN
-F 2 "" H 2200 3750 60  0000 C CNN
-F 3 "" H 2200 3750 60  0000 C CNN
-	1    2200 3750
-	1    0    0    -1
+P 2250 3700
+F 0 "D3" H 2250 3800 40  0000 C CNN
+F 1 "D_Schottky" H 2250 3600 40  0000 C CNN
+F 2 "" H 2250 3700 60  0000 C CNN
+F 3 "" H 2250 3700 60  0000 C CNN
+	1    2250 3700
+	0    1    1    0
 $EndComp
-Wire Wire Line
-	2400 3750 2400 4050
-Wire Wire Line
-	2450 3900 2400 3900
-Connection ~ 2400 3900
 $Comp
 L +2.8VD #PWR177
@@
 Wire Wire Line
 	1800 3700 1800 4050
-Wire Wire Line
-	1650 4050 2050 4050
 Connection ~ 1800 4050
-Wire Wire Line
-	2000 3750 2000 3400
-Connection ~ 2000 3400
-$Comp
-L D_Schottky D2
-U 1 1 54152FCC
-P 2250 5350
-F 0 "D2" H 2250 5450 40  0000 C CNN
-F 1 "D_Schottky" H 2250 5250 40  0000 C CNN
-F 2 "" H 2250 5350 60  0000 C CNN
-F 3 "" H 2250 5350 60  0000 C CNN
-	1    2250 5350
-	1    0    0    -1
-$EndComp
 $Comp
 L D_Schottky D1
 U 1 1 54152FD2
-P 2250 5050
-F 0 "D1" H 2250 5150 40  0000 C CNN
-F 1 "D_Schottky" H 2250 4950 40  0000 C CNN
-F 2 "" H 2250 5050 60  0000 C CNN
-F 3 "" H 2250 5050 60  0000 C CNN
-	1    2250 5050
-	1    0    0    -1
+P 2250 5000
+F 0 "D1" H 2250 5100 40  0000 C CNN
+F 1 "D_Schottky" H 2250 4900 40  0000 C CNN
+F 2 "" H 2250 5000 60  0000 C CNN
+F 3 "" H 2250 5000 60  0000 C CNN
+	1    2250 5000
+	0    1    1    0
 $EndComp
-Wire Wire Line
-	2450 5050 2450 5350
-Wire Wire Line
-	2500 5200 2450 5200
-Connection ~ 2450 5200
 $Comp
 L PMOS_SOT Q5
@@
 	0    -1   -1   0
 $EndComp
-$Comp
-L R R84
-U 1 1 54152FE7
-P 1550 5350
-F 0 "R84" V 1630 5350 40  0000 C CNN
-F 1 "100k" V 1557 5351 40  0000 C CNN
-F 2 "" V 1480 5350 30  0000 C CNN
-F 3 "" H 1550 5350 30  0000 C CNN
-	1    1550 5350
-	0    1    1    0
-$EndComp
 Wire Wire Line
 	1350 4700 1600 4700
 Wire Wire Line
 	2000 4700 3400 4700
-Wire Wire Line
-	1850 5000 1850 5350
-Wire Wire Line
-	1700 5350 2100 5350
-Connection ~ 1850 5350
-Wire Wire Line
-	2050 5050 2050 4700
-Connection ~ 2050 4700
-$Comp
-L GND #PWR175
-U 1 1 5415334A
-P 1300 5350
-F 0 "#PWR175" H 1300 5350 30  0001 C CNN
-F 1 "GND" H 1300 5280 30  0001 C CNN
-F 2 "" H 1300 5350 60  0000 C CNN
-F 3 "" H 1300 5350 60  0000 C CNN
-	1    1300 5350
-	0    1    1    0
-$EndComp
 $Comp
 L PWR_FLAG #FLG1
@@
 L +3V3 #PWR193
 U 1 1 54E828E9
-P 2500 5200
-F 0 "#PWR193" H 2500 5050 60  0001 C CNN
-F 1 "+3V3" H 2500 5340 60  0000 C CNN
-F 2 "" H 2500 5200 60  0000 C CNN
-F 3 "" H 2500 5200 60  0000 C CNN
-	1    2500 5200
-	0    1    1    0
+P 2050 5350
+F 0 "#PWR193" H 2050 5200 60  0001 C CNN
+F 1 "+3V3" H 2050 5490 60  0000 C CNN
+F 2 "" H 2050 5350 60  0000 C CNN
+F 3 "" H 2050 5350 60  0000 C CNN
+	1    2050 5350
+	-1   0    0    1
 $EndComp
 $Comp
 L +3V3 #PWR191
 U 1 1 54E82D16
-P 2450 3900
-F 0 "#PWR191" H 2450 3750 60  0001 C CNN
-F 1 "+3V3" H 2450 4040 60  0000 C CNN
-F 2 "" H 2450 3900 60  0000 C CNN
-F 3 "" H 2450 3900 60  0000 C CNN
-	1    2450 3900
+P 2450 4050
+F 0 "#PWR191" H 2450 3900 60  0001 C CNN
+F 1 "+3V3" H 2450 4190 60  0000 C CNN
+F 2 "" H 2450 4050 60  0000 C CNN
+F 3 "" H 2450 4050 60  0000 C CNN
+	1    2450 4050
 	0    1    1    0
 $EndComp
-Wire Wire Line
-	2400 3750 2350 3750
-Wire Wire Line
-	2050 3750 2000 3750
-Wire Wire Line
-	2400 4050 2350 4050
-Wire Wire Line
-	1400 5350 1300 5350
-Wire Wire Line
-	2100 5050 2050 5050
-Wire Wire Line
-	2450 5050 2400 5050
-Wire Wire Line
-	2450 5350 2400 5350
 Connection ~ 3250 5200
 Wire Wire Line
@@
 Wire Wire Line
 	1350 4050 1250 4050
+Wire Wire Line
+	2250 4850 2250 4700
+Connection ~ 2250 4700
+Wire Wire Line
+	2250 5300 2250 5150
+Wire Wire Line
+	1850 5300 2250 5300
+Wire Wire Line
+	1850 5300 1850 5000
+Connection ~ 2050 5300
+Wire Wire Line
+	2050 5350 2050 5300
+Wire Wire Line
+	2250 4050 2250 3850
+Wire Wire Line
+	1650 4050 2450 4050
+Wire Wire Line
+	2250 3550 2250 3400
+Connection ~ 2250 3400
+Connection ~ 2250 4050
 $EndSCHEMATC

Commit message: Charger short circuit fix. Capacitor optimizations.
Parts:
- removed C103, C107, C114, C122, C86, C87, C88, C96: 10uF, symbol C_Small
- removed C90, C91: 100nF, symbol C_Small
- C102, C106, C108, C44, C45, C52, C53, C59, C60, C61, C67, C68, C75, C76, C80, C81, C97: value 10uF -> 1uF
- C66, C82: value 10uF -> 100nF
- C74: value 10uF -> 100pF
- C85: value 100nF -> 100pF
Connections:
- wire segments 214 -> 308
Other:
- note removed: "CARD READER"
- moved on the sheet: R70

Commit message: Reverse diode fix. Cap changes.
Parts:
- removed C123: 10uF, symbol C_Small
- C108: value 1uF -> 1uF 10V
- C115, C116, C119: value 10uF -> 10uF 10V
- C62: value PAS311HR-VA6R -> EEEFTA471XAP
Connections:
- wire segments 308 -> 199
Other:
- note added: "RTC for 5 minutes\nwithout battery"
- note removed: "SUPERCAP\nRTC for 2 hours\nwithout battery"

Commit message: Footprints, LC filter
Parts:
- removed C69: 1uF, symbol C_Small
- removed C73: 100nF, symbol C_Small
- added C86: 10uF, symbol C_Small
- added L6: 4.7uH, symbol INDUCTOR_SMALL
- C100, C101, C102, C104, C105, C106, C108, C109, C110, C112, C113, C117, C118, C120, C121, C124, C125, C127, C130, C131, C44, C45, C46, C47, C48, C52, C53, C54, C55, C56, C57, C58, C59, C60, C61, C63, C64, C65, C66, C67, C68, C70, C71, C72, C74, C75, C76, C77, C78, C79, C80, C81, C82, C83, C84, C85, C89, C94, C95, C97, C99: footprint (none) -> Capacitors_SMD:C_0402
- C111, C115, C116, C119, C126, C128, C129, C43, C49, C50, C51, C92, C93, C98: footprint (none) -> Capacitors_SMD:C_0603
Connections:
- wire segments 199 -> 198

Commit message: Reorder RC cap. Remove holter-rescue library.
Connections:
- wire segments 198 -> 304
Other:
- moved on the sheet: C62

Commit message: More footprints.
Parts:
- C86: footprint (none) -> Capacitors_SMD:C_0603
- R63, R64, R65, R66, R67, R68, R69, R70, R71, R72, R73, R74, R75, R76, R77: footprint (none) -> Resistors_SMD:R_0402
- U24, U25, U26: footprint (none) -> Housings_SOT-23_SOT-143_TSOT-6:SOT-23-6
- U27: footprint (none) -> TO_SOT_Packages_SMD:SOT-23-5
Connections:
- wire segments 304 -> 198
Other:
- moved on the sheet: C62

Commit message: More footprints.
Parts:
- C62: value EEEFTA471XAP -> TPSC337M006R0080
- L1, L2, L3: value 4.7uH -> 4.7uH PFL2015-472MEC; footprint (none) -> Capacitors_SMD:C_0805
- L6: footprint (none) -> Capacitors_SMD:C_0805
Changed lines of the file:
@@
 EESchema Schematic File Version 2
-LIBS:holter-rescue
 LIBS:power
 LIBS:device
@@
 P 1850 2400
 F 0 "L2" H 1850 2500 50  0000 C CNN
-F 1 "4.7uH" H 1850 2350 50  0000 C CNN
-F 2 "" H 1850 2400 60  0001 C CNN
+F 1 "4.7uH PFL2015-472MEC" H 1850 2600 50  0000 C CNN
+F 2 "Capacitors_SMD:C_0805" H 1850 2400 60  0001 C CNN
 F 3 "" H 1850 2400 60  0000 C CNN
 	1    1850 2400
@@
 P 1850 1400
 F 0 "L1" H 1850 1500 50  0000 C CNN
-F 1 "4.7uH" H 1850 1350 50  0000 C CNN
-F 2 "" H 1850 1400 60  0001 C CNN
+F 1 "4.7uH PFL2015-472MEC" H 1850 1600 50  0000 C CNN
+F 2 "Capacitors_SMD:C_0805" H 1850 1400 60  0001 C CNN
 F 3 "" H 1850 1400 60  0000 C CNN
 	1    1850 1400
@@
 P 6100 2200
 F 0 "L3" H 6100 2300 50  0000 C CNN
-F 1 "4.7uH" H 6100 2150 50  0000 C CNN
-F 2 "" H 6100 2200 60  0001 C CNN
+F 1 "4.7uH PFL2015-472MEC" H 6150 2400 50  0000 C CNN
+F 2 "Capacitors_SMD:C_0805" H 6100 2200 60  0001 C CNN
 F 3 "" H 6100 2200 60  0000 C CNN
 	1    6100 2200
@@
 P 3750 3800
 F 0 "C62" V 3700 3850 40  0000 L CNN
-F 1 "EEEFTA471XAP" V 3900 3550 40  0000 L CNN
+F 1 "TPSC337M006R0080" H 3800 3650 40  0000 L CNN
 F 2 "" H 3788 3650 30  0001 C CNN
 F 3 "" H 3750 3800 60  0000 C CNN
@@
 F 0 "L6" H 8900 2300 50  0000 C CNN
 F 1 "4.7uH" H 8900 2150 50  0000 C CNN
-F 2 "" H 8900 2200 60  0001 C CNN
+F 2 "Capacitors_SMD:C_0805" H 8900 2200 60  0001 C CNN
 F 3 "" H 8900 2200 60  0000 C CNN
 	1    8900 2200
