File: Hardware/power.sch (KiCad schematic (older format))
At the start: 117 parts, among them P3 BAT+, P4 BAT-, Q1 SI1403, Q2 SI1403, Q3 SI1403, Q4 SI1403, Q5 SI1403, U24 TLV61220, U25 TLV61220, U26 TLV61220, U27 LM3671, U28 DS2710

Commit message: Fixed ADS1298 library.
Changed lines of the file:
@@
 EESchema Schematic File Version 2
+LIBS:holter-rescue
 LIBS:power
 LIBS:device
@@
 LIBS:rgbled
 LIBS:lis2dh12
+LIBS:holter-cache
 EELAYER 25 0
 EELAYER END
@@
 	1    0    0    -1
 $EndComp
+$Comp
+L PWR_FLAG #FLG0274
+U 1 1 56189D0A
+P 9400 2200
+F 0 "#FLG0274" H 9400 2295 30  0001 C CNN
+F 1 "PWR_FLAG" H 9400 2380 30  0000 C CNN
+F 2 "" H 9400 2200 60  0000 C CNN
+F 3 "" H 9400 2200 60  0000 C CNN
+	1    9400 2200
+	1    0    0    -1
+$EndComp

Commit message: More footprints.
Parts:
- L5: footprint (none) -> Capacitors_SMD:C_0805
- Q1, Q2, Q3, Q4, Q5: footprint SC70-3 -> (none)
Changed lines of the file:
@@
 F 0 "L5" H 7800 1550 50  0000 C CNN
 F 1 "2.2uH" H 7800 1400 50  0000 C CNN
-F 2 "" H 7800 1450 60  0001 C CNN
+F 2 "Capacitors_SMD:C_0805" H 7800 1450 60  0001 C CNN
 F 3 "" H 7800 1450 60  0000 C CNN
 	1    7800 1450
@@
 F 0 "Q3" V 7000 3800 40  0000 R CNN
 F 1 "SI1403" V 7350 3750 40  0000 R CNN
-F 2 "SC70-3" H 6900 3750 29  0001 C CNN
+F 2 "" H 6900 3750 29  0001 C CNN
 F 3 "" H 7100 3650 60  0000 C CNN
 	1    7100 3650
@@
 F 0 "Q2" V 5550 4600 40  0000 R CNN
 F 1 "SI1403" V 5900 4550 40  0000 R CNN
-F 2 "SC70-3" H 5450 4550 29  0001 C CNN
+F 2 "" H 5450 4550 29  0001 C CNN
 F 3 "" H 5650 4450 60  0000 C CNN
 	1    5650 4450
@@
 F 0 "Q1" V 3500 4950 40  0000 R CNN
 F 1 "SI1403" V 3850 4900 40  0000 R CNN
-F 2 "SC70-3" H 3400 4900 29  0001 C CNN
+F 2 "" H 3400 4900 29  0001 C CNN
 F 3 "" H 3600 4800 60  0000 C CNN
 	1    3600 4800
@@
 F 0 "Q4" V 1650 3650 40  0000 R CNN
 F 1 "SI1403" V 2000 3600 40  0000 R CNN
-F 2 "SC70-3" H 1550 3600 29  0001 C CNN
+F 2 "" H 1550 3600 29  0001 C CNN
 F 3 "" H 1750 3500 60  0000 C CNN
 	1    1750 3500
@@
 F 0 "Q5" V 1700 4950 40  0000 R CNN
 F 1 "SI1403" V 2050 4900 40  0000 R CNN
-F 2 "SC70-3" H 1600 4900 29  0001 C CNN
+F 2 "" H 1600 4900 29  0001 C CNN
 F 3 "" H 1800 4800 60  0000 C CNN
 	1    1800 4800

Commit message: Footprints...
Parts:
- Q1, Q2, Q3, Q4, Q5: value SI1403 -> PMF170XP
- U28: footprint (none) -> Footprints:T1034N1

Commit message: Footprints.
Parts:
- L4: value 15uH -> 15uH SLF7055T-150M2R1-3PF; footprint (none) -> Footprints:SLF7055
- Q1, Q2, Q3, Q4, Q5: footprint (none) -> TO_SOT_Packages_SMD:SC-70
Changed lines of the file:
@@
 F 0 "Q3" V 7000 3800 40  0000 R CNN
 F 1 "PMF170XP" V 7350 3750 40  0000 R CNN
-F 2 "" H 6900 3750 29  0001 C CNN
+F 2 "TO_SOT_Packages_SMD:SC-70" H 6900 3750 29  0001 C CNN
 F 3 "" H 7100 3650 60  0000 C CNN
 	1    7100 3650
@@
 U 1 1 54108602
 P 8000 3550
-F 0 "L4" H 8000 3650 50  0000 C CNN
-F 1 "15uH" H 8000 3500 50  0000 C CNN
-F 2 "" H 8000 3550 60  0001 C CNN
+F 0 "L4" H 8000 3500 50  0000 C CNN
+F 1 "15uH SLF7055T-150M2R1-3PF" H 8050 3700 50  0000 C CNN
+F 2 "Footprints:SLF7055" H 8000 3550 60  0001 C CNN
 F 3 "" H 8000 3550 60  0000 C CNN
 	1    8000 3550
@@
 F 0 "Q2" V 5550 4600 40  0000 R CNN
 F 1 "PMF170XP" V 5900 4550 40  0000 R CNN
-F 2 "" H 5450 4550 29  0001 C CNN
+F 2 "TO_SOT_Packages_SMD:SC-70" H 5450 4550 29  0001 C CNN
 F 3 "" H 5650 4450 60  0000 C CNN
 	1    5650 4450
@@
 F 0 "Q1" V 3500 4950 40  0000 R CNN
 F 1 "PMF170XP" V 3850 4900 40  0000 R CNN
-F 2 "" H 3400 4900 29  0001 C CNN
+F 2 "TO_SOT_Packages_SMD:SC-70" H 3400 4900 29  0001 C CNN
 F 3 "" H 3600 4800 60  0000 C CNN
 	1    3600 4800
@@
 F 0 "Q4" V 1650 3650 40  0000 R CNN
 F 1 "PMF170XP" V 2000 3600 40  0000 R CNN
-F 2 "" H 1550 3600 29  0001 C CNN
+F 2 "TO_SOT_Packages_SMD:SC-70" H 1550 3600 29  0001 C CNN
 F 3 "" H 1750 3500 60  0000 C CNN
 	1    1750 3500
@@
 F 0 "Q5" V 1700 4950 40  0000 R CNN
 F 1 "PMF170XP" V 2050 4900 40  0000 R CNN
-F 2 "" H 1600 4900 29  0001 C CNN
+F 2 "TO_SOT_Packages_SMD:SC-70" H 1600 4900 29  0001 C CNN
 F 3 "" H 1800 4800 60  0000 C CNN
 	1    1800 4800

Commit message: Footprints.
Parts:
- removed D8: D_Schottky, symbol D_Schottky
- C62: footprint (none) -> Capacitors_Tantalum_SMD:TantalC_SizeC_EIA-6032_Reflow
- D1, D3, D4: value D_Schottky -> DB2S20500L; footprint (none) -> Diodes_SMD:SOD-323
- D7: footprint (none) -> Diodes_SMD:SOD-123
- Q3: value PMF170XP -> NTR4101PT1G; footprint TO_SOT_Packages_SMD:SC-70 -> TO_SOT_Packages_SMD:SOT-23
- Rsense1: footprint (none) -> Capacitors_SMD:C_0805
Connections:
- wire segments 198 -> 197

Commit message: Footprints.
Parts:
- removed P3: BAT+, symbol CONN_01X01
- added D2: D_Schottky, Diodes_SMD:SOD-123, symbol D_Schottky
Connections:
- net labels added: BAT+
- wire segments 197 -> 198
Changed lines of the file:
@@
-$EndComp
-$Comp
-L CONN_01X01 P3
-U 1 1 54E8133C
-P 10050 4250
-F 0 "P3" H 10050 4350 50  0000 C CNN
-F 1 "BAT+" V 10150 4250 50  0000 C CNN
-F 2 "" H 10050 4250 60  0001 C CNN
-F 3 "" H 10050 4250 60  0000 C CNN
-	1    10050 4250
-	1    0    0    -1
 $EndComp
 $Comp
@@
 	7300 3550 7750 3550
 Connection ~ 7500 3550
-Wire Wire Line
-	8250 3550 9350 3550
 Connection ~ 8450 3550
 Connection ~ 8700 3550
@@
 	8300 4250 8850 4250
 Wire Wire Line
-	9150 4250 9850 4250
+	9150 4250 10150 4250
 Wire Wire Line
 	9150 4500 9850 4500
@@
 	8450 3600 8450 3550
 Wire Wire Line
-	8700 3600 8700 3550
+	8700 3550 8700 3600
 Wire Wire Line
 	8450 3900 8450 3950
@@
 	1    0    0    -1
 $EndComp
+$Comp
+L D_Schottky D2
+U 1 1 561FEE35
+P 9050 3550
+F 0 "D2" H 9050 3650 40  0000 C CNN
+F 1 "D_Schottky" H 9050 3450 40  0000 C CNN
+F 2 "Diodes_SMD:SOD-123" H 9050 3550 60  0001 C CNN
+F 3 "" H 9050 3550 60  0000 C CNN
+	1    9050 3550
+	-1   0    0    1
+$EndComp
+Wire Wire Line
+	8250 3550 8900 3550
+Wire Wire Line
+	9200 3550 9350 3550
+Text Label 10150 4250 2    60   ~ 0
+BAT+
 $EndSCHEMATC

Commit message: Footprints.
Parts:
- TH1: footprint (none) -> Resistors_ThroughHole:Resistor_Horizontal_RM10mm
