File: Hardware/power.sch (KiCad schematic (older format))
At the start: 91 parts, among them M1 USB_Power_Module, P4 BAT-, Q1 PMF170XP, Q4 PMF170XP, Q5 PMF170XP, U24 TLV61220, U25 TLV61220, U26 TLV61220

Commit message: Placement + additional bypass capacitors.
Parts:
- removed C98: 10uF, Capacitors_SMD:C_0603, symbol C_Small
- added C1234: 22uF, Capacitors_SMD:C_0805, symbol C_Small
- added C_LSH1, C_LSH2: 100nF, Capacitors_SMD:C_0402, symbol C_Small
- C51: value 10uF -> 22uF
Changed lines of the file:
@@
 ECG VDD
-$Comp
-L C_Small C98
-U 1 1 5410D17B
-P 4350 7350
-F 0 "C98" H 4375 7400 30  0000 L CNN
-F 1 "10uF" H 4375 7300 30  0000 L CNN
-F 2 "Capacitors_SMD:C_0603" H 4350 7350 60  0001 C CNN
-F 3 "" H 4350 7350 60  0000 C CNN
-	1    4350 7350
-	1    0    0    -1
-$EndComp
 $Comp
 L C_Small C101
@@
 P 4550 7350
 F 0 "C51" H 4575 7400 30  0000 L CNN
-F 1 "10uF" H 4575 7300 30  0000 L CNN
+F 1 "22uF" H 4575 7300 30  0000 L CNN
 F 2 "Capacitors_SMD:C_0603" H 4550 7350 60  0001 C CNN
 F 3 "" H 4550 7350 60  0000 C CNN
@@
 Wire Wire Line
 	4150 7250 5350 7250
-Connection ~ 4350 7250
 Wire Wire Line
 	2200 2700 2100 2700
@@
 	5050 6150 5550 6150
 Connection ~ 5300 6150
-Connection ~ 4350 7450
 Connection ~ 4550 7450
 Connection ~ 4550 7250
@@
 	8000 4000 8000 4100
 Connection ~ 8250 4100
+$Comp
+L C_Small C1234
+U 1 1 562AE305
+P 8250 4200
+F 0 "C1234" H 8275 4250 30  0000 L CNN
+F 1 "22uF" H 8275 4150 30  0000 L CNN
+F 2 "Capacitors_SMD:C_0805" H 8250 4200 60  0001 C CNN
+F 3 "" H 8250 4200 60  0000 C CNN
+	1    8250 4200
+	1    0    0    -1
+$EndComp
+$Comp
+L GND #PWR0265
+U 1 1 562AE9B6
+P 8250 4300
+F 0 "#PWR0265" H 8250 4300 30  0001 C CNN
+F 1 "GND" H 8250 4230 30  0001 C CNN
+F 2 "" H 8250 4300 60  0000 C CNN
+F 3 "" H 8250 4300 60  0000 C CNN
+	1    8250 4300
+	1    0    0    -1
+$EndComp
+$Comp
+L C_Small C_LSH1
+U 1 1 562B4986
+P 3550 6800
+F 0 "C_LSH1" H 3575 6850 30  0000 L CNN
+F 1 "100nF" H 3575 6750 30  0000 L CNN
+F 2 "Capacitors_SMD:C_0402" H 3550 6800 60  0001 C CNN
+F 3 "" H 3550 6800 60  0000 C CNN
+	1    3550 6800
+	1    0    0    -1
+$EndComp
+$Comp
+L GND #PWR?
+U 1 1 562B4E7B
+P 3550 6900
+F 0 "#PWR?" H 3550 6900 30  0001 C CNN
+F 1 "GND" H 3550 6830 30  0001 C CNN
+F 2 "" H 3550 6900 60  0000 C CNN
+F 3 "" H 3550 6900 60  0000 C CNN
+	1    3550 6900
+	1    0    0    -1
+$EndComp
+$Comp
+L +1V8 #PWR?
+U 1 1 562B4F9A
+P 3550 6700
+F 0 "#PWR?" H 3550 6550 60  0001 C CNN
+F 1 "+1V8" H 3550 6840 60  0000 C CNN
+F 2 "" H 3550 6700 60  0000 C CNN
+F 3 "" H 3550 6700 60  0000 C CNN
+	1    3550 6700
+	1    0    0    -1
+$EndComp
+$Comp
+L C_Small C_LSH2
+U 1 1 562B59BF
+P 3550 6250
+F 0 "C_LSH2" H 3575 6300 30  0000 L CNN
+F 1 "100nF" H 3575 6200 30  0000 L CNN
+F 2 "Capacitors_SMD:C_0402" H 3550 6250 60  0001 C CNN
+F 3 "" H 3550 6250 60  0000 C CNN
+	1    3550 6250
+	1    0    0    -1
+$EndComp
+$Comp
+L GND #PWR?
+U 1 1 562B6134
+P 3550 6350
+F 0 "#PWR?" H 3550 6350 30  0001 C CNN
+F 1 "GND" H 3550 6280 30  0001 C CNN
+F 2 "" H 3550 6350 60  0000 C CNN
+F 3 "" H 3550 6350 60  0000 C CNN
+	1    3550 6350
+	1    0    0    -1
+$EndComp
+$Comp
+L +3V3 #PWR?
+U 1 1 562B63CA
+P 3550 6150
+F 0 "#PWR?" H 3550 6000 60  0001 C CNN
+F 1 "+3V3" H 3550 6290 60  0000 C CNN
+F 2 "" H 3550 6150 60  0000 C CNN
+F 3 "" H 3550 6150 60  0000 C CNN
+	1    3550 6150
+	1    0    0    -1
+$EndComp
 $EndSCHEMATC

Commit message: Removed unnecessary bypass capacitors.
Parts:
- removed C106, C68, C76, C81: 1uF, Capacitors_SMD:C_0402, symbol C_Small
- removed C117, C72, C79, C84: 100nF, Capacitors_SMD:C_0402, symbol C_Small
Connections:
- wire segments 151 -> 143
Changed lines of the file:
@@
-$EndComp
-$Comp
-L C_Small C68
-U 1 1 5410C521
-P 2300 7350
-F 0 "C68" H 2325 7400 30  0000 L CNN
-F 1 "1uF" H 2325 7300 30  0000 L CNN
-F 2 "Capacitors_SMD:C_0402" H 2300 7350 60  0001 C CNN
-F 3 "" H 2300 7350 60  0000 C CNN
-	1    2300 7350
-	1    0    0    -1
-$EndComp
-$Comp
-L C_Small C72
-U 1 1 5410C528
-P 2500 7350
-F 0 "C72" H 2525 7400 30  0000 L CNN
-F 1 "100nF" H 2525 7300 30  0000 L CNN
-F 2 "Capacitors_SMD:C_0402" H 2500 7350 60  0001 C CNN
-F 3 "" H 2500 7350 60  0000 C CNN
-	1    2500 7350
-	1    0    0    -1
-$EndComp
-$Comp
-L C_Small C76
-U 1 1 5410C52F
-P 2800 7350
-F 0 "C76" H 2825 7400 30  0000 L CNN
-F 1 "1uF" H 2825 7300 30  0000 L CNN
-F 2 "Capacitors_SMD:C_0402" H 2800 7350 60  0001 C CNN
-F 3 "" H 2800 7350 60  0000 C CNN
-	1    2800 7350
-	1    0    0    -1
-$EndComp
-$Comp
-L C_Small C79
-U 1 1 5410C536
-P 3000 7350
-F 0 "C79" H 3025 7400 30  0000 L CNN
-F 1 "100nF" H 3025 7300 30  0000 L CNN
-F 2 "Capacitors_SMD:C_0402" H 3000 7350 60  0001 C CNN
-F 3 "" H 3000 7350 60  0000 C CNN
-	1    3000 7350
-	1    0    0    -1
-$EndComp
-$Comp
-L C_Small C81
-U 1 1 5410C53D
-P 3300 7350
-F 0 "C81" H 3325 7400 30  0000 L CNN
-F 1 "1uF" H 3325 7300 30  0000 L CNN
-F 2 "Capacitors_SMD:C_0402" H 3300 7350 60  0001 C CNN
-F 3 "" H 3300 7350 60  0000 C CNN
-	1    3300 7350
-	1    0    0    -1
-$EndComp
-$Comp
-L C_Small C84
-U 1 1 5410C544
-P 3500 7350
-F 0 "C84" H 3525 7400 30  0000 L CNN
-F 1 "100nF" H 3525 7300 30  0000 L CNN
-F 2 "Capacitors_SMD:C_0402" H 3500 7350 60  0001 C CNN
-F 3 "" H 3500 7350 60  0000 C CNN
-	1    3500 7350
-	1    0    0    -1
 $EndComp
 $Comp
@@
 	1    0    0    -1
 $EndComp
-$Comp
-L GND #PWR0196
-U 1 1 5410C567
-P 2400 7500
-F 0 "#PWR0196" H 2400 7500 30  0001 C CNN
-F 1 "GND" H 2400 7430 30  0001 C CNN
-F 2 "" H 2400 7500 60  0000 C CNN
-F 3 "" H 2400 7500 60  0000 C CNN
-	1    2400 7500
-	1    0    0    -1
-$EndComp
-$Comp
-L GND #PWR0197
-U 1 1 5410C56D
-P 2900 7500
-F 0 "#PWR0197" H 2900 7500 30  0001 C CNN
-F 1 "GND" H 2900 7430 30  0001 C CNN
-F 2 "" H 2900 7500 60  0000 C CNN
-F 3 "" H 2900 7500 60  0000 C CNN
-	1    2900 7500
-	1    0    0    -1
-$EndComp
-$Comp
-L GND #PWR0198
-U 1 1 5410C573
-P 3400 7500
-F 0 "#PWR0198" H 3400 7500 30  0001 C CNN
-F 1 "GND" H 3400 7430 30  0001 C CNN
-F 2 "" H 3400 7500 60  0000 C CNN
-F 3 "" H 3400 7500 60  0000 C CNN
-	1    3400 7500
-	1    0    0    -1
-$EndComp
 Text Notes 900  7200 0    39   ~ 0
 ECG VAA
@@
 CPU
 $Comp
-L C_Small C106
-U 1 1 5410D0E5
+L C_Small C109
+U 1 1 5410D0EC
 P 4300 6800
-F 0 "C106" H 4325 6850 30  0000 L CNN
-F 1 "1uF" H 4325 6750 30  0000 L CNN
+F 0 "C109" H 4325 6850 30  0000 L CNN
+F 1 "100nF" H 4325 6750 30  0000 L CNN
 F 2 "Capacitors_SMD:C_0402" H 4300 6800 60  0001 C CNN
 F 3 "" H 4300 6800 60  0000 C CNN
@@
 $EndComp
 $Comp
-L C_Small C109
-U 1 1 5410D0EC
-P 4500 6800
-F 0 "C109" H 4525 6850 30  0000 L CNN
-F 1 "100nF" H 4525 6750 30  0000 L CNN
-F 2 "Capacitors_SMD:C_0402" H 4500 6800 60  0001 C CNN
-F 3 "" H 4500 6800 60  0000 C CNN
-	1    4500 6800
-	1    0    0    -1
-$EndComp
-$Comp
-L C_Small C117
-U 1 1 5410D0FA
-P 4900 6800
-F 0 "C117" H 4925 6850 30  0000 L CNN
-F 1 "100nF" H 4925 6750 30  0000 L CNN
-F 2 "Capacitors_SMD:C_0402" H 4900 6800 60  0001 C CNN
-F 3 "" H 4900 6800 60  0000 C CNN
-	1    4900 6800
-	1    0    0    -1
-$EndComp
-$Comp
-L C_Small C124
-U 1 1 5410D108
-P 5150 6800
-F 0 "C124" H 5175 6850 30  0000 L CNN
-F 1 "100nF" H 5175 6750 30  0000 L CNN
-F 2 "Capacitors_SMD:C_0402" H 5150 6800 60  0001 C CNN
-F 3 "" H 5150 6800 60  0000 C CNN
-	1    5150 6800
-	1    0    0    -1
-$EndComp
-$Comp
 L GND #PWR0204
 U 1 1 5410D10F
-P 4400 6950
-F 0 "#PWR0204" H 4400 6950 30  0001 C CNN
-F 1 "GND" H 4400 6880 30  0001 C CNN
-F 2 "" H 4400 6950 60  0000 C CNN
-F 3 "" H 4400 6950 60  0000 C CNN
-	1    4400 6950
+P 4300 6950
+F 0 "#PWR0204" H 4300 6950 30  0001 C CNN
+F 1 "GND" H 4300 6880 30  0001 C CNN
+F 2 "" H 4300 6950 60  0000 C CNN
+F 3 "" H 4300 6950 60  0000 C CNN
+	1    4300 6950
 	1    0    0    -1
 $EndComp
@@
 L GND #PWR0205
 U 1 1 5410D115
-P 4900 6950
-F 0 "#PWR0205" H 4900 6950 30  0001 C CNN
-F 1 "GND" H 4900 6880 30  0001 C CNN
-F 2 "" H 4900 6950 60  0000 C CNN
-F 3 "" H 4900 6950 60  0000 C CNN
-	1    4900 6950
-	1    0    0    -1
-$EndComp
-$Comp
-L GND #PWR0206
-U 1 1 5410D11B
-P 5150 6950
-F 0 "#PWR0206" H 5150 6950 30  0001 C CNN
-F 1 "GND" H 5150 6880 30  0001 C CNN
-F 2 "" H 5150 6950 60  0000 C CNN
-F 3 "" H 5150 6950 60  0000 C CNN
-	1    5150 6950
+P 4500 6950
+F 0 "#PWR0205" H 4500 6950 30  0001 C CNN
+F 1 "GND" H 4500 6880 30  0001 C CNN
+F 2 "" H 4500 6950 60  0000 C CNN
+F 3 "" H 4500 6950 60  0000 C CNN
+	1    4500 6950
 	1    0    0    -1
 $EndComp
@@
 	1300 7450 1500 7450
 Wire Wire Line
-	3300 7450 3500 7450
-Wire Wire Line
-	3400 7500 3400 7450
-Connection ~ 3400 7450
-Wire Wire Line
-	2800 7450 3000 7450
-Wire Wire Line
-	2900 7500 2900 7450
-Connection ~ 2900 7450
-Wire Wire Line
-	2300 7450 2500 7450
-Wire Wire Line
-	2400 7450 2400 7500
-Connection ~ 2400 7450
-Wire Wire Line
 	1800 7450 2000 7450
 Wire Wire Line
@@
 	1400 7500 1400 7450
 Connection ~ 1400 7450
-Connection ~ 3300 7250
-Connection ~ 3000 7250
-Connection ~ 2800 7250
-Connection ~ 2500 7250
-Connection ~ 2300 7250
 Connection ~ 2000 7250
 Connection ~ 1800 7250
@@
 Connection ~ 800  6700
 Wire Wire Line
-	5150 6950 5150 6900
-Wire Wire Line
-	4900 6950 4900 6900
-Wire Wire Line
-	4300 6900 4500 6900
-Wire Wire Line
-	4400 6950 4400 6900
-Connection ~ 4400 6900
-Wire Wire Line
-	4300 6700 5150 6700
+	4500 6950 4500 6900
 Wire Wire Line
 	6300 6900 6500 6900
@@
 Connection ~ 5800 6700
 Connection ~ 4300 6700
-Connection ~ 4500 6700
-Connection ~ 4900 6700
 Wire Wire Line
 	4150 7450 4750 7450
@@
 Connection ~ 2250 3400
 Connection ~ 2250 4050
-Wire Wire Line
-	800  7250 3500 7250
 Wire Wire Line
 	4150 6350 4650 6350
@@
 $EndComp
 $Comp
-L GND #PWR?
+L GND #PWR0266
 U 1 1 562B4E7B
 P 3550 6900
-F 0 "#PWR?" H 3550 6900 30  0001 C CNN
+F 0 "#PWR0266" H 3550 6900 30  0001 C CNN
 F 1 "GND" H 3550 6830 30  0001 C CNN
 F 2 "" H 3550 6900 60  0000 C CNN
@@
 $EndComp
 $Comp
-L +1V8 #PWR?
+L +1V8 #PWR0267
 U 1 1 562B4F9A
 P 3550 6700
-F 0 "#PWR?" H 3550 6550 60  0001 C CNN
+F 0 "#PWR0267" H 3550 6550 60  0001 C CNN
 F 1 "+1V8" H 3550 6840 60  0000 C CNN
 F 2 "" H 3550 6700 60  0000 C CNN
@@
 $EndComp
 $Comp
-L GND #PWR?
+L GND #PWR0268
 U 1 1 562B6134
 P 3550 6350
-F 0 "#PWR?" H 3550 6350 30  0001 C CNN
+F 0 "#PWR0268" H 3550 6350 30  0001 C CNN
 F 1 "GND" H 3550 6280 30  0001 C CNN
 F 2 "" H 3550 6350 60  0000 C CNN
@@
 $EndComp
 $Comp
-L +3V3 #PWR?
+L +3V3 #PWR0269
 U 1 1 562B63CA
 P 3550 6150
-F 0 "#PWR?" H 3550 6000 60  0001 C CNN
+F 0 "#PWR0269" H 3550 6000 60  0001 C CNN
 F 1 "+3V3" H 3550 6290 60  0000 C CNN
 F 2 "" H 3550 6150 60  0000 C CNN
@@
 	1    0    0    -1
 $EndComp
+$Comp
+L C_Small C124
+U 1 1 5410D108
+P 4500 6800
+F 0 "C124" H 4525 6850 30  0000 L CNN
+F 1 "100nF" H 4525 6750 30  0000 L CNN
+F 2 "Capacitors_SMD:C_0402" H 4500 6800 60  0001 C CNN
+F 3 "" H 4500 6800 60  0000 C CNN
+	1    4500 6800
+	1    0    0    -1
+$EndComp
+Wire Wire Line
+	4300 6950 4300 6900
+Wire Wire Line
+	4500 6700 4300 6700
+Wire Wire Line
+	800  7250 2000 7250
 $EndSCHEMATC

Commit message: Fixed ADS1298 footprint. Routing of the analog parts.
Parts:
- removed C102: 1uF, Capacitors_SMD:C_0402, symbol C_Small
- removed C104: 100nF, Capacitors_SMD:C_0402, symbol C_Small
Connections:
- wire segments 143 -> 141

Commit message: More traces.
Parts:
- added C_ADC1: 100nF, Capacitors_SMD:C_0402, symbol C_Small
Changed lines of the file:
@@
 	4500 6950 4500 6900
 Wire Wire Line
-	5800 6900 6000 6900
+	5800 6900 6300 6900
 Wire Wire Line
 	5900 6950 5900 6900
@@
 	800  7250 2000 7250
 Wire Wire Line
-	6000 6700 5800 6700
+	5800 6700 6300 6700
 Wire Wire Line
 	6800 5100 8550 5100
 Wire Wire Line
 	6800 5100 6800 5000
+$Comp
+L C_Small C_ADC1
+U 1 1 562E4539
+P 6300 6800
+F 0 "C_ADC1" H 6325 6850 30  0000 L CNN
+F 1 "100nF" H 6325 6750 30  0000 L CNN
+F 2 "Capacitors_SMD:C_0402" H 6300 6800 60  0001 C CNN
+F 3 "" H 6300 6800 60  0000 C CNN
+	1    6300 6800
+	1    0    0    -1
+$EndComp
+Connection ~ 6000 6900
+Connection ~ 6000 6700
 $EndSCHEMATC

Commit message: Rearrangement of CPU pins, even more traces, fixed LGA footprint
Parts:
- removed C83: 100nF, Capacitors_SMD:C_0402, symbol C_Small
Connections:
- wire segments 141 -> 140
Changed lines of the file:
@@
-$EndComp
-$Comp
-L C_Small C83
-U 1 1 5413DB26
-P 2400 6250
-F 0 "C83" H 2425 6300 30  0000 L CNN
-F 1 "100nF" H 2425 6200 30  0000 L CNN
-F 2 "Capacitors_SMD:C_0402" H 2400 6250 60  0001 C CNN
-F 3 "" H 2400 6250 60  0000 C CNN
-	1    2400 6250
-	1    0    0    -1
 $EndComp
 $Comp
@@
 $Comp
 L GND #PWR0242
-U 1 1 5617798D
-P 2400 6400
-F 0 "#PWR0242" H 2400 6400 30  0001 C CNN
-F 1 "GND" H 2400 6330 30  0001 C CNN
-F 2 "" H 2400 6400 60  0000 C CNN
-F 3 "" H 2400 6400 60  0000 C CNN
-	1    2400 6400
-	1    0    0    -1
-$EndComp
-$Comp
-L GND #PWR0243
 U 1 1 56177AFA
 P 2700 6400
-F 0 "#PWR0243" H 2700 6400 30  0001 C CNN
+F 0 "#PWR0242" H 2700 6400 30  0001 C CNN
 F 1 "GND" H 2700 6330 30  0001 C CNN
 F 2 "" H 2700 6400 60  0000 C CNN
@@
 $EndComp
 $Comp
-L GND #PWR0244
+L GND #PWR0243
 U 1 1 56177C67
 P 3000 6400
-F 0 "#PWR0244" H 3000 6400 30  0001 C CNN
+F 0 "#PWR0243" H 3000 6400 30  0001 C CNN
 F 1 "GND" H 3000 6330 30  0001 C CNN
 F 2 "" H 3000 6400 60  0000 C CNN
@@
 $EndComp
 $Comp
-L GND #PWR0245
+L GND #PWR0244
 U 1 1 5614D7DF
 P 9400 2650
-F 0 "#PWR0245" H 9400 2650 30  0001 C CNN
+F 0 "#PWR0244" H 9400 2650 30  0001 C CNN
 F 1 "GND" H 9400 2580 30  0001 C CNN
 F 2 "" H 9400 2650 60  0000 C CNN
@@
 $EndComp
 $Comp
-L PWR_FLAG #FLG0246
+L PWR_FLAG #FLG0245
 U 1 1 56189D0A
 P 9400 2200
-F 0 "#FLG0246" H 9400 2295 30  0001 C CNN
+F 0 "#FLG0245" H 9400 2295 30  0001 C CNN
 F 1 "PWR_FLAG" H 9400 2380 30  0000 C CNN
 F 2 "" H 9400 2200 60  0000 C CNN
@@
 $EndComp
 $Comp
-L GND #PWR0247
+L GND #PWR0246
 U 1 1 5624848D
 P 4800 2900
-F 0 "#PWR0247" H 4800 2900 30  0001 C CNN
+F 0 "#PWR0246" H 4800 2900 30  0001 C CNN
 F 1 "GND" H 4800 2830 30  0001 C CNN
 F 2 "" H 4800 2900 60  0000 C CNN
@@
 $EndComp
 $Comp
-L PWR_FLAG #FLG0248
+L PWR_FLAG #FLG0247
 U 1 1 5624ACE6
 P 4800 2400
-F 0 "#FLG0248" H 4800 2495 30  0001 C CNN
+F 0 "#FLG0247" H 4800 2495 30  0001 C CNN
 F 1 "PWR_FLAG" H 4800 2580 30  0000 C CNN
 F 2 "" H 4800 2400 60  0000 C CNN
@@
 $EndComp
 $Comp
-L PWR_FLAG #FLG0249
+L PWR_FLAG #FLG0248
 U 1 1 54143E48
 P 8400 4100
-F 0 "#FLG0249" H 8400 4195 30  0001 C CNN
+F 0 "#FLG0248" H 8400 4195 30  0001 C CNN
 F 1 "PWR_FLAG" H 8400 4280 30  0000 C CNN
 F 2 "" H 8400 4100 60  0000 C CNN
@@
 $EndComp
 $Comp
-L VCC #PWR0250
+L VCC #PWR0249
 U 1 1 541107D7
 P 8250 4100
-F 0 "#PWR0250" H 8250 4200 30  0001 C CNN
+F 0 "#PWR0249" H 8250 4200 30  0001 C CNN
 F 1 "VCC" H 8250 4200 30  0000 C CNN
 F 2 "" H 8250 4100 60  0000 C CNN
@@
 $EndComp
 $Comp
-L GND #PWR0251
+L GND #PWR0250
 U 1 1 541130D3
 P 8350 5400
-F 0 "#PWR0251" H 8350 5400 30  0001 C CNN
+F 0 "#PWR0250" H 8350 5400 30  0001 C CNN
 F 1 "GND" H 8350 5330 30  0001 C CNN
 F 2 "" H 8350 5400 60  0000 C CNN
@@
 	2100 6400 2100 6350
 Wire Wire Line
-	2400 6400 2400 6350
-Wire Wire Line
 	2700 6350 2700 6400
 Wire Wire Line
@@
 Connection ~ 1800 6150
 Connection ~ 2100 6150
-Connection ~ 2400 6150
 Connection ~ 2700 6150
 Connection ~ 4150 7250
@@
 $EndComp
 $Comp
-L GND #PWR0252
+L GND #PWR0251
 U 1 1 562D076C
 P 6800 5600
-F 0 "#PWR0252" H 6800 5600 30  0001 C CNN
+F 0 "#PWR0251" H 6800 5600 30  0001 C CNN
 F 1 "GND" H 6800 5530 30  0001 C CNN
 F 2 "" H 6800 5600 60  0000 C CNN
@@
 Connection ~ 6800 3550
 $Comp
-L +5V #PWR0253
+L +5V #PWR0252
 U 1 1 562D2FDE
 P 6800 3300
-F 0 "#PWR0253" H 6800 3150 50  0001 C CNN
+F 0 "#PWR0252" H 6800 3150 50  0001 C CNN
 F 1 "+5V" H 6800 3440 50  0000 C CNN
 F 2 "" H 6800 3300 60  0000 C CNN
@@
 	6800 4300 7700 4300
 $Comp
-L +2.8VD #PWR0254
+L +2.8VD #PWR0253
 U 1 1 562D5EF8
 P 6800 4200
-F 0 "#PWR0254" H 6800 4160 30  0001 C CNN
+F 0 "#PWR0253" H 6800 4160 30  0001 C CNN
 F 1 "+2.8VD" H 6800 4310 30  0000 C CNN
 F 2 "" H 6800 4200 60  0000 C CNN
@@
 	6800 4000 8000 4000
 $Comp
-L VBAT #PWR0255
+L VBAT #PWR0254
 U 1 1 562D661F
 P 7700 3900
-F 0 "#PWR0255" H 7700 3860 30  0001 C CNN
+F 0 "#PWR0254" H 7700 3860 30  0001 C CNN
 F 1 "VBAT" H 7700 4010 30  0000 C CNN
 F 2 "" H 7700 3900 60  0000 C CNN
@@
 $EndComp
 $Comp
-L +3V3 #PWR0256
+L +3V3 #PWR0255
 U 1 1 562DC84B
 P 7700 4300
-F 0 "#PWR0256" H 7700 4150 60  0001 C CNN
+F 0 "#PWR0255" H 7700 4150 60  0001 C CNN
 F 1 "+3V3" H 7700 4440 60  0000 C CNN
 F 2 "" H 7700 4300 60  0000 C CNN
@@
 $EndComp
 $Comp
-L PWR_FLAG #FLG0257
+L PWR_FLAG #FLG0256
 U 1 1 562DD352
 P 7450 4300
-F 0 "#FLG0257" H 7450 4395 30  0001 C CNN
+F 0 "#FLG0256" H 7450 4395 30  0001 C CNN
 F 1 "PWR_FLAG" H 7450 4480 30  0000 C CNN
 F 2 "" H 7450 4300 60  0000 C CNN
@@
 	7700 3900 6800 3900
 $Comp
-L PWR_FLAG #FLG0258
+L PWR_FLAG #FLG0257
 U 1 1 562DE072
 P 7450 3900
-F 0 "#FLG0258" H 7450 3995 30  0001 C CNN
+F 0 "#FLG0257" H 7450 3995 30  0001 C CNN
 F 1 "PWR_FLAG" H 7450 4080 30  0000 C CNN
 F 2 "" H 7450 3900 60  0000 C CNN
@@
 $EndComp
 $Comp
-L GND #PWR0259
+L GND #PWR0258
 U 1 1 562AE9B6
 P 8250 4300
-F 0 "#PWR0259" H 8250 4300 30  0001 C CNN
+F 0 "#PWR0258" H 8250 4300 30  0001 C CNN
 F 1 "GND" H 8250 4230 30  0001 C CNN
 F 2 "" H 8250 4300 60  0000 C CNN
@@
 $EndComp
 $Comp
-L GND #PWR0260
+L GND #PWR0259
 U 1 1 562B4E7B
 P 3550 6900
-F 0 "#PWR0260" H 3550 6900 30  0001 C CNN
+F 0 "#PWR0259" H 3550 6900 30  0001 C CNN
 F 1 "GND" H 3550 6830 30  0001 C CNN
 F 2 "" H 3550 6900 60  0000 C CNN
@@
 $EndComp
 $Comp
-L +1V8 #PWR0261
+L +1V8 #PWR0260
 U 1 1 562B4F9A
 P 3550 6700
-F 0 "#PWR0261" H 3550 6550 60  0001 C CNN
+F 0 "#PWR0260" H 3550 6550 60  0001 C CNN
 F 1 "+1V8" H 3550 6840 60  0000 C CNN
 F 2 "" H 3550 6700 60  0000 C CNN
@@
 $EndComp
 $Comp
-L GND #PWR0262
+L GND #PWR0261
 U 1 1 562B6134
 P 3550 6350
-F 0 "#PWR0262" H 3550 6350 30  0001 C CNN
+F 0 "#PWR0261" H 3550 6350 30  0001 C CNN
 F 1 "GND" H 3550 6280 30  0001 C CNN
 F 2 "" H 3550 6350 60  0000 C CNN
@@
 $EndComp
 $Comp
-L +3V3 #PWR0263
+L +3V3 #PWR0262
 U 1 1 562B63CA
 P 3550 6150
-F 0 "#PWR0263" H 3550 6000 60  0001 C CNN
+F 0 "#PWR0262" H 3550 6000 60  0001 C CNN
 F 1 "+3V3" H 3550 6290 60  0000 C CNN
 F 2 "" H 3550 6150 60  0000 C CNN

Commit message: Everything is connected on the main board.
Parts:
- C125: value 100nF -> 47uF; footprint Capacitors_SMD:C_0402 -> Capacitors_SMD:C_1206
