File: Hardware/_autosave-holter.kicad_pcb (KiCad board)
At the start: 2 copper layers, 33.5 x 48 mm, 270 parts, among them CN1 2TAP, CN2 2TAP, CN3 3TAP, IC1 256kx8, M1 USB_Power_Module, M2 USB_Power_Module, P1 CONN_01X07, P2 PROG, P3 SCREW, P4 BAT-, Q1 PMF170XP, Q2 PMF170XP, Q3 NTR4101PT1G, Q4 PMF170XP, Q5 PMF170XP, U1 TXB0106, U10 TS5A3159, U11 TS5A3159, U12 ESD_PROTECTOR, U13 ESD_PROTECTOR, U14 ESD_PROTECTOR, U15 ESD_PROTECTOR, U16 ESD_PROTECTOR, U17 ESD_PROTECTOR, U18 ESD_PROTECTOR, U19 ESD_PROTECTOR, U2 TXB0106, U20 ESD_PROTECTOR, U21 ESD_PROTECTOR, U22 ESD_PROTECTOR, U23 ESD_PROTECTOR, U24 TLV61220, U25 TLV61220, U26 TLV61220, U27 LM3671, U28 DS2710, U29 LIS2DH12, U3 TiWi-uB2, U4 STM32F4x1_64, U5 uSD, U6 ADS1298, U7 USBULC6-2M6, U8 USB2641, U9 OPA379, X1 32768, Y1 24 MHz, Y2 10 MHz

Commit message: Placement of parts.
Parts:
- moved C43 17.4 mm to (65.5, 89.4)
- moved U1 7.53 mm to (78.4, 68.6)
- moved C98 3.39 mm to (85.8, 74.5)
Changed lines of the file:
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@@
   )
   (module Capacitors_SMD:C_0603 (layer F.Cu)
-    (at 77.5 76.8 90)
+    (at 65.5 89.375 90)
     (descr "Capacitor SMD 0603, reflow soldering, AVX (see smccp.pdf)")
     (tags "capacitor 0603")
@@
   )
   (module Capacitors_SMD:C_0603 (layer F.Cu)
-    (at 88.9 75.9)
+    (at 85.8 74.525)
     (descr "Capacitor SMD 0603, reflow soldering, AVX (see smccp.pdf)")
     (tags "capacitor 0603")
@@
   )
   (module Footprints:RGY16 (layer F.Cu)
-    (at 84.8 72.625)
+    (at 78.425 68.625)
     (fp_text reference U1 (at 0 3.52) (layer F.SilkS)
       (effects (font (size 1 1) (thickness 0.15)))
