File: Hardware/usb_power.sch (KiCad schematic (older format))
At the start: 30 parts, among them M2 USB_Power_Module, Q2 PMF170XP, Q3 NTR4101PT1G, U27 LM3671, U28 DS2710

Commit message: Routing attempt.
Connections:
- wire segments 71 -> 70
Changed lines of the file:
@@
 $EndComp
 $Comp
-L PWR_FLAG #FLG0265
+L PWR_FLAG #FLG0264
 U 1 1 562B9127
 P 6700 3300
-F 0 "#FLG0265" H 6700 3395 30  0001 C CNN
+F 0 "#FLG0264" H 6700 3395 30  0001 C CNN
 F 1 "PWR_FLAG" H 6700 3480 30  0000 C CNN
 F 2 "" H 6700 3300 60  0000 C CNN
@@
 $EndComp
 $Comp
-L GNDPWR #PWR0266
+L GNDPWR #PWR0265
 U 1 1 562BDA3A
 P 2200 5200
-F 0 "#PWR0266" H 2200 5000 50  0001 C CNN
+F 0 "#PWR0265" H 2200 5000 50  0001 C CNN
 F 1 "GNDPWR" H 2200 5070 50  0000 C CNN
 F 2 "" H 2200 5150 60  0000 C CNN
@@
 $EndComp
 $Comp
-L GNDPWR #PWR0267
+L GNDPWR #PWR0266
 U 1 1 562BDADC
 P 9050 3500
-F 0 "#PWR0267" H 9050 3300 50  0001 C CNN
+F 0 "#PWR0266" H 9050 3300 50  0001 C CNN
 F 1 "GNDPWR" H 9050 3370 50  0000 C CNN
 F 2 "" H 9050 3450 60  0000 C CNN
@@
 $EndComp
 $Comp
-L GNDPWR #PWR0268
+L GNDPWR #PWR0267
 U 1 1 562BDB23
 P 8600 3700
-F 0 "#PWR0268" H 8600 3500 50  0001 C CNN
+F 0 "#PWR0267" H 8600 3500 50  0001 C CNN
 F 1 "GNDPWR" H 8600 3570 50  0000 C CNN
 F 2 "" H 8600 3650 60  0000 C CNN
@@
 $EndComp
 $Comp
-L GNDPWR #PWR0269
+L GNDPWR #PWR0268
 U 1 1 562BDBBC
 P 7250 4200
-F 0 "#PWR0269" H 7250 4000 50  0001 C CNN
+F 0 "#PWR0268" H 7250 4000 50  0001 C CNN
 F 1 "GNDPWR" H 7450 4150 50  0000 C CNN
 F 2 "" H 7250 4150 60  0000 C CNN
@@
 $EndComp
 $Comp
-L GNDPWR #PWR0270
+L GNDPWR #PWR0269
 U 1 1 562BDC03
 P 7000 4200
-F 0 "#PWR0270" H 7000 4000 50  0001 C CNN
+F 0 "#PWR0269" H 7000 4000 50  0001 C CNN
 F 1 "GNDPWR" H 7000 4070 50  0000 C CNN
 F 2 "" H 7000 4150 60  0000 C CNN
@@
 $EndComp
 $Comp
-L GNDPWR #PWR0271
+L GNDPWR #PWR0270
 U 1 1 562BDCEC
 P 6450 3950
-F 0 "#PWR0271" H 6450 3750 50  0001 C CNN
+F 0 "#PWR0270" H 6450 3750 50  0001 C CNN
 F 1 "GNDPWR" H 6450 3800 50  0000 C CNN
 F 2 "" H 6450 3900 60  0000 C CNN
@@
 $EndComp
 $Comp
-L GNDPWR #PWR0272
+L GNDPWR #PWR0271
 U 1 1 562BDD33
 P 6200 3950
-F 0 "#PWR0272" H 6200 3750 50  0001 C CNN
+F 0 "#PWR0271" H 6200 3750 50  0001 C CNN
 F 1 "GNDPWR" H 6100 3800 50  0000 C CNN
 F 2 "" H 6200 3900 60  0000 C CNN
@@
 $EndComp
 $Comp
-L GNDPWR #PWR0273
+L GNDPWR #PWR0272
 U 1 1 562BDE80
 P 6700 2900
-F 0 "#PWR0273" H 6700 2700 50  0001 C CNN
+F 0 "#PWR0272" H 6700 2700 50  0001 C CNN
 F 1 "GNDPWR" H 6700 2770 50  0000 C CNN
 F 2 "" H 6700 2850 60  0000 C CNN
@@
 $EndComp
 $Comp
-L GNDPWR #PWR0274
+L GNDPWR #PWR0273
 U 1 1 562BDEC7
 P 6950 2900
-F 0 "#PWR0274" H 6950 2700 50  0001 C CNN
+F 0 "#PWR0273" H 6950 2700 50  0001 C CNN
 F 1 "GNDPWR" H 7050 2750 50  0000 C CNN
 F 2 "" H 6950 2850 60  0000 C CNN
@@
 $EndComp
 $Comp
-L GNDPWR #PWR0275
+L GNDPWR #PWR0274
 U 1 1 562BE364
 P 7800 2900
-F 0 "#PWR0275" H 7800 2700 50  0001 C CNN
+F 0 "#PWR0274" H 7800 2700 50  0001 C CNN
 F 1 "GNDPWR" H 7550 2850 50  0000 C CNN
 F 2 "" H 7800 2850 60  0000 C CNN
@@
 $EndComp
 $Comp
-L GNDPWR #PWR0276
+L GNDPWR #PWR0275
 U 1 1 562BE3FD
 P 8750 2900
-F 0 "#PWR0276" H 8750 2700 50  0001 C CNN
+F 0 "#PWR0275" H 8750 2700 50  0001 C CNN
 F 1 "GNDPWR" H 8750 2770 50  0000 C CNN
 F 2 "" H 8750 2850 60  0000 C CNN
@@
 $EndComp
 $Comp
-L GNDPWR #PWR0277
+L GNDPWR #PWR0276
 U 1 1 562BE444
 P 9000 2900
-F 0 "#PWR0277" H 9000 2700 50  0001 C CNN
+F 0 "#PWR0276" H 9000 2700 50  0001 C CNN
 F 1 "GNDPWR" H 9200 2850 50  0000 C CNN
 F 2 "" H 9000 2850 60  0000 C CNN
@@
 $EndComp
 $Comp
-L +5P #PWR0278
+L +5P #PWR0277
 U 1 1 562BF0F2
 P 6500 2500
-F 0 "#PWR0278" H 6500 2350 50  0001 C CNN
+F 0 "#PWR0277" H 6500 2350 50  0001 C CNN
 F 1 "+5P" H 6500 2640 50  0000 C CNN
 F 2 "" H 6500 2500 60  0000 C CNN
@@
 $EndComp
 $Comp
-L +5P #PWR0279
+L +5P #PWR0278
 U 1 1 562BF140
 P 5600 3300
-F 0 "#PWR0279" H 5600 3150 50  0001 C CNN
+F 0 "#PWR0278" H 5600 3150 50  0001 C CNN
 F 1 "+5P" H 5600 3440 50  0000 C CNN
 F 2 "" H 5600 3300 60  0000 C CNN
@@
 $EndComp
 $Comp
-L +5P #PWR0280
+L +5P #PWR0279
 U 1 1 562BF187
 P 8050 3050
-F 0 "#PWR0280" H 8050 2900 50  0001 C CNN
+F 0 "#PWR0279" H 8050 2900 50  0001 C CNN
 F 1 "+5P" H 8050 3190 50  0000 C CNN
 F 2 "" H 8050 3050 60  0000 C CNN
@@
 $EndComp
 $Comp
-L +5P #PWR0281
+L +5P #PWR0280
 U 1 1 562BF5F4
 P 2800 3100
-F 0 "#PWR0281" H 2800 2950 50  0001 C CNN
+F 0 "#PWR0280" H 2800 2950 50  0001 C CNN
 F 1 "+5P" H 2800 3240 50  0000 C CNN
 F 2 "" H 2800 3100 60  0000 C CNN
@@
 RTC for 5 minutes\nwithout battery
 $Comp
-L PWR_FLAG #FLG0282
+L PWR_FLAG #FLG0281
 U 1 1 562C7273
 P 3700 3750
-F 0 "#FLG0282" H 3700 3845 30  0001 C CNN
+F 0 "#FLG0281" H 3700 3845 30  0001 C CNN
 F 1 "PWR_FLAG" H 3700 3930 30  0000 C CNN
 F 2 "" H 3700 3750 60  0000 C CNN
@@
 BAT+
 $Comp
-L GNDPWR #PWR0283
+L GNDPWR #PWR0282
 U 1 1 562C7921
 P 3900 4150
-F 0 "#PWR0283" H 3900 3950 50  0001 C CNN
+F 0 "#PWR0282" H 3900 3950 50  0001 C CNN
 F 1 "GNDPWR" H 3900 4020 50  0000 C CNN
 F 2 "" H 3900 4100 60  0000 C CNN
@@
 $EndComp
 $Comp
-L PWR_FLAG #FLG0284
+L PWR_FLAG #FLG0283
 U 1 1 562C8C8E
 P 9350 5350
-F 0 "#FLG0284" H 9350 5445 30  0001 C CNN
+F 0 "#FLG0283" H 9350 5445 30  0001 C CNN
 F 1 "PWR_FLAG" H 9350 5530 30  0000 C CNN
 F 2 "" H 9350 5350 60  0000 C CNN
@@
 	7400 5550 7200 5550
 $Comp
-L +3.3VP #PWR0285
+L +3.3VP #PWR0284
 U 1 1 562C8DDB
 P 2650 3850
-F 0 "#PWR0285" H 2800 3800 50  0001 C CNN
+F 0 "#PWR0284" H 2800 3800 50  0001 C CNN
 F 1 "+3.3VP" V 2650 4050 50  0000 C CNN
 F 2 "" H 2650 3850 60  0000 C CNN
@@
 $EndComp
 $Comp
-L +3.3VP #PWR0286
+L +3.3VP #PWR0285
 U 1 1 562C9056
 P 9450 5350
-F 0 "#PWR0286" H 9600 5300 50  0001 C CNN
+F 0 "#PWR0285" H 9600 5300 50  0001 C CNN
 F 1 "+3.3VP" H 9450 5450 50  0000 C CNN
 F 2 "" H 9450 5350 60  0000 C CNN
@@
 $EndComp
 $Comp
-L +5P #PWR0287
+L +5P #PWR0286
 U 1 1 562C9638
 P 6400 5350
-F 0 "#PWR0287" H 6400 5200 50  0001 C CNN
+F 0 "#PWR0286" H 6400 5200 50  0001 C CNN
 F 1 "+5P" H 6400 5490 50  0000 C CNN
 F 2 "" H 6400 5350 60  0000 C CNN
@@
 $EndComp
 $Comp
-L GNDPWR #PWR0288
+L GNDPWR #PWR0287
 U 1 1 562C970D
 P 6500 5550
-F 0 "#PWR0288" H 6500 5350 50  0001 C CNN
+F 0 "#PWR0287" H 6500 5350 50  0001 C CNN
 F 1 "GNDPWR" H 6400 5400 50  0000 C CNN
 F 2 "" H 6500 5500 60  0000 C CNN
@@
 $EndComp
 $Comp
-L GNDPWR #PWR0289
+L GNDPWR #PWR0288
 U 1 1 562C976C
 P 6700 5550
-F 0 "#PWR0289" H 6700 5350 50  0001 C CNN
+F 0 "#PWR0288" H 6700 5350 50  0001 C CNN
 F 1 "GNDPWR" H 6750 5400 50  0000 C CNN
 F 2 "" H 6700 5500 60  0000 C CNN
@@
 $EndComp
 $Comp
-L GNDPWR #PWR0290
+L GNDPWR #PWR0289
 U 1 1 562C9864
 P 7400 5450
-F 0 "#PWR0290" H 7400 5250 50  0001 C CNN
+F 0 "#PWR0289" H 7400 5250 50  0001 C CNN
 F 1 "GNDPWR" H 7100 5300 50  0000 C CNN
 F 2 "" H 7400 5400 60  0000 C CNN
@@
 EN_3V3
 $Comp
-L GNDPWR #PWR0291
+L GNDPWR #PWR0290
 U 1 1 562CA0C1
 P 9150 5550
-F 0 "#PWR0291" H 9150 5350 50  0001 C CNN
+F 0 "#PWR0290" H 9150 5350 50  0001 C CNN
 F 1 "GNDPWR" H 9050 5400 50  0000 C CNN
 F 2 "" H 9150 5500 60  0000 C CNN
@@
 $EndComp
 $Comp
-L GNDPWR #PWR0292
+L GNDPWR #PWR0291
 U 1 1 562CA19A
 P 9350 5550
-F 0 "#PWR0292" H 9350 5350 50  0001 C CNN
+F 0 "#PWR0291" H 9350 5350 50  0001 C CNN
 F 1 "GNDPWR" H 9450 5400 50  0000 C CNN
 F 2 "" H 9350 5500 60  0000 C CNN
@@
 Text Label 2700 4350 2    60   ~ 0
 EN_3V3
-Wire Wire Line
-	2200 4550 2200 4650
-Wire Wire Line
-	2200 4650 2750 4650
-Text Label 2750 4650 2    60   ~ 0
+Text Label 2750 4550 2    60   ~ 0
 BAT-
 Connection ~ 9650 3200
@@
 $EndComp
 $Comp
-L GNDPWR #PWR0293
+L GNDPWR #PWR0292
 U 1 1 562DB395
 P 9000 4550
-F 0 "#PWR0293" H 9000 4350 50  0001 C CNN
+F 0 "#PWR0292" H 9000 4350 50  0001 C CNN
 F 1 "GNDPWR" H 9000 4420 50  0000 C CNN
 F 2 "" H 9000 4500 60  0000 C CNN
@@
 	9000 4050 8750 4050
 $Comp
-L PWR_FLAG #FLG0294
+L PWR_FLAG #FLG0293
 U 1 1 562DE658
 P 2200 4900
-F 0 "#FLG0294" H 2200 4995 30  0001 C CNN
+F 0 "#FLG0293" H 2200 4995 30  0001 C CNN
 F 1 "PWR_FLAG" H 2200 5080 30  0000 C CNN
 F 2 "" H 2200 4900 60  0000 C CNN
@@
 	2200 3100 2200 3200
 $Comp
-L PWR_FLAG #FLG0295
+L PWR_FLAG #FLG0294
 U 1 1 562DEDBD
 P 2500 3100
-F 0 "#FLG0295" H 2500 3195 30  0001 C CNN
+F 0 "#FLG0294" H 2500 3195 30  0001 C CNN
 F 1 "PWR_FLAG" H 2500 3280 30  0000 C CNN
 F 2 "" H 2500 3100 60  0000 C CNN
@@
 Connection ~ 7300 5550
 $Comp
-L GNDPWR #PWR0296
+L GNDPWR #PWR0295
 U 1 1 562E070E
 P 7300 5850
-F 0 "#PWR0296" H 7300 5650 50  0001 C CNN
+F 0 "#PWR0295" H 7300 5650 50  0001 C CNN
 F 1 "GNDPWR" H 7300 5720 50  0000 C CNN
 F 2 "" H 7300 5800 60  0000 C CNN
@@
 $EndComp
 $Comp
-L GNDPWR #PWR0297
+L GNDPWR #PWR0296
 U 1 1 5627CE4B
 P 7350 3400
-F 0 "#PWR0297" H 7350 3200 50  0001 C CNN
+F 0 "#PWR0296" H 7350 3200 50  0001 C CNN
 F 1 "GNDPWR" V 7350 3150 50  0000 C CNN
 F 2 "" H 7350 3350 60  0000 C CNN
@@
 	0    1    1    0
 $EndComp
+Wire Wire Line
+	2200 4550 2750 4550
 $EndSCHEMATC

Commit message: New footprint for the inductor of the charger.
Parts:
- L4: value 15uH SLF7055T-150M2R1-3PF -> 15uH SRR6038; footprint Footprints:SLF7055 -> Footprints:SRR6038
Changed lines of the file:
@@
 P 8300 2500
 F 0 "L4" H 8300 2450 50  0000 C CNN
-F 1 "15uH SLF7055T-150M2R1-3PF" H 8350 2650 50  0000 C CNN
-F 2 "Footprints:SLF7055" H 8300 2500 60  0001 C CNN
+F 1 "15uH SRR6038" H 8350 2650 50  0000 C CNN
+F 2 "Footprints:SRR6038" H 8300 2500 60  0001 C CNN
 F 3 "" H 8300 2500 60  0000 C CNN
 	1    8300 2500

Commit message: Schematic fixes.
Parts:
- M2: value USB_Power_Module -> ECG mainboard
Connections:
- wire segments 70 -> 93
Other:
- moved on the sheet: C108, C112, C116, C120, C126, C127, C62, L4, L5, Q2, Q3, R3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
